Commit message: Remove unsupported args

File: description/robots/lbr4.robot.xacro (robot description, xacro)
@@ -1,5 +1,5 @@
 <?xml version="1.0" ?>
 <robot xmlns:xacro="http://www.ros.org/wiki/xacro" name="lbr4">
-  <xacro:arg name="end_effector"      default="None"  /> <!-- [allegro, reflex, push_stick, rigid_obj] -->
+  <xacro:arg name="end_effector"      default="None"  /> <!-- [reflex, push_stick, rigid_obj] -->
   <xacro:arg name="ft_sensor"         default="true" />
   <xacro:arg name="robot_table"       default="false" />
@@ -8,5 +8,4 @@
   <xacro:arg name="robot_name"        default="lbr4"  />
   <xacro:arg name="control"           default="false" />
-  <xacro:arg name="biotac"            default="true" />
   <xacro:arg name="actuate_reflex"    default="false" />
   <xacro:arg name="gazebo"            default="false"  />
@@ -73,20 +72,4 @@
       <xacro:arg name="robot_name" value="$(arg robot_name)"/>
     </xacro:include>
-  </xacro:if>
-  <!-- Allegro hand -->
-  <xacro:if value="${end_effector == 'allegro'}">
-    <xacro:include filename="$(find description)/robots/allegro.robot.xacro">
-      <xacro:arg name="gazebo" value="$(arg gazebo)"/>
-      <xacro:arg name="control" value="$(arg control)"/>
-      <xacro:arg name="biotac" value="$(arg biotac)"/>
-    </xacro:include>
-    <!-- Include the KUKA mount -->
-    <xacro:include filename="${urdf_path}/mounts/lbr4_mount.urdf.xacro"/>
-    <xacro:lbr4_mount parent="${ee_mount_frame}"/>
-    <joint name="lbr4_allegro" type="fixed">
-      <parent link="lbr4_mount"/>
-      <child link="allegro_mount"/>
-      <origin xyz="-0.0 0 -0.0" rpy="0 1.57 0"/>
-    </joint>
   </xacro:if>
   <!-- ReFlex Hand -->

File: description/robots/optoforce.robot.xacro (robot description, xacro)
@@ -1,5 +1,5 @@
 <?xml version="1.0" ?>
 <robot xmlns:xacro="http://www.ros.org/wiki/xacro" name="lbr4">
-  <xacro:arg name="end_effector" default="None"  doc="[biotac_hold, push_stick,cube]"/>
+  <xacro:arg name="end_effector" default="None"  doc="[push_stick,cube]"/>
   <xacro:arg name="gazebo"       default="false"  />
   <!-- ========================================================================================== -->
@@ -47,13 +47,4 @@
     </joint>
   </xacro:if>
-  <xacro:if value="${end_effector == 'biotac_mount'}">
-    <xacro:include filename="${urdf_path}/end_effectors/biotac_mount.urdf.xacro"/>
-    <xacro:biotac_mount/>
-    <joint name="optoforce_to_biotac_mount" type="fixed">
-	<origin xyz="0 0 0.05" rpy="0 0 0"/>
-	<parent link="optoforce_model_link"/>
-      <child link="biotac_mount_link" />
-    </joint>
-  </xacro:if>
   <xacro:if value="${end_effector == 'cube'}">
     <xacro:include filename="${urdf_path}/end_effectors/cube.urdf.xacro"/>
