Commit message: Fix Gazebo warning about missing color

File: description/urdf/reflex/reflex.urdf.xacro (robot description, xacro)
@@ -1,5 +1,5 @@
 <?xml version="1.0"?>
 <robot xmlns:xacro="http://www.ros.org/wiki/xacro" name="reflex">
-  <xacro:arg name="actuate_reflex"             default="true"/>
+  <xacro:arg name="actuate_reflex" default="true"/>
   <xacro:arg name="use_reflex_contact_sensors" default="true"/>
   <!-- Switch joint type for actuated joints depending on if they are being used for control -->
@@ -13,4 +13,16 @@
   <xacro:property name="mesh_path" value="package://description/meshes/reflex"/>
   <xacro:include filename="$(find description)/urdf/xacro_macros/inertia_tensors.xacro"/>
+  <!-- ===================================== MATERIALS ======================================= -->
+  <!-- Gazebo won't be able to read these colors but they are required RViz
+  see this issue https://robotics.stackexchange.com/questions/20506/gazebo-not-reading-the-material-color-in-urdf -->
+  <material name="black">
+    <color rgba="0 0 0 0"/>
+  </material>
+  <material name="dark_grey">
+    <color rgba="0.2 0.2 0.2 1"/>
+  </material>
+  <material name="gold">
+    <color rgba="${254/255} ${216/255} ${93/255} 1"/>
+  </material>
   <!-- ======================================= Masses ======================================== -->
   <!-- These are rough approximations, the total hand mass was measured to be about 0.9kg,     -->
@@ -18,12 +30,12 @@
   <!-- is being given to shell/pad, treating fingers as almost massless, so that KDL chain for -->
   <!-- arm can just go through the palm pad and be accounting for most of the hand mass.       -->
-  <xacro:property name="flex_link_mass"     value="0.01"/>
+  <xacro:property name="flex_link_mass" value="0.01"/>
   <xacro:property name="proximal_link_mass" value="0.01"/>
-  <xacro:property name="distal_link_mass"   value="0.01"/>
-  <xacro:property name="proximal_pad_mass"  value="0.01"/>
-  <xacro:property name="distal_pad_mass"    value="0.01"/>
-  <xacro:property name="swivel_link_mass"   value="0.01"/>
-  <xacro:property name="shell_mass"         value="0.74"/>
-  <xacro:property name="pad_mass"           value="0.1"/>
+  <xacro:property name="distal_link_mass" value="0.01"/>
+  <xacro:property name="proximal_pad_mass" value="0.01"/>
+  <xacro:property name="distal_pad_mass" value="0.01"/>
+  <xacro:property name="swivel_link_mass" value="0.01"/>
+  <xacro:property name="shell_mass" value="0.74"/>
+  <xacro:property name="pad_mass" value="0.1"/>
   <!-- ====================================== Link Macros ==================================== -->
   <xacro:macro name="flex_link" params="finger_id">
@@ -32,20 +44,18 @@
         <origin xyz="0.0005 0 -0.003" rpy="0 0 0"/>
         <geometry>
-	  <box size="0.017 0.014 0.0065"/>
-        </geometry>
-	<material name="gold">
-	  <color rgba="${254/255} ${216/255} ${93/255} 1"/>
-	</material>
-      </visual>
-      <inertial>
-        <origin xyz="0 0 0" rpy="0 0 0"/>
-	<mass value="${flex_link_mass}"/>
-	<xacro:cuboid_inertia m="${flex_link_mass}" x="0.005" y="0.014" z="0.015"/>
-      </inertial>
-      <collision>
-        <origin xyz="0 0 0" rpy="0 0 0"/>
-  	<geometry>
-	  <box size="0.01 0.01 0.01"/>
-  	</geometry>
+          <box size="0.017 0.014 0.0065"/>
+        </geometry>
+        <material name="gold"/>
+      </visual>
+      <inertial>
+        <origin xyz="0 0 0" rpy="0 0 0"/>
+        <mass value="${flex_link_mass}"/>
+        <xacro:cuboid_inertia m="${flex_link_mass}" x="0.005" y="0.014" z="0.015"/>
+      </inertial>
+      <collision>
+        <origin xyz="0 0 0" rpy="0 0 0"/>
+        <geometry>
+          <box size="0.01 0.01 0.01"/>
+        </geometry>
       </collision>
     </link>
@@ -54,20 +64,20 @@
     <link name="proximal_${finger_id}">
       <visual>
-	<origin xyz="-0.011 0.007 0.011" rpy="${pi} 0 0"/>
-	<geometry>
+        <origin xyz="-0.011 0.007 0.011" rpy="${pi} 0 0"/>
+        <geometry>
           <mesh filename="${mesh_path}/proximal.STL"/>
-	</geometry>
-	<material name="black"/>
-      </visual>
-      <inertial>
-	<origin xyz="-0.011 0.007 0.011" rpy="${pi} 0 0"/>
-	<mass value="${proximal_link_mass}"/>
-	<xacro:cuboid_inertia m="${proximal_link_mass}" x="0.02" y="0.15" z="0.071"/>
-      </inertial>
-      <collision>
-	<origin xyz="-0.011 0.007 0.011" rpy="${pi} 0 0"/>
-	<geometry>
-	  <mesh filename="${mesh_path}/proximal_coll.STL"/>
-	</geometry>
+        </geometry>
+        <material name="black"/>
+      </visual>
+      <inertial>
+        <origin xyz="-0.011 0.007 0.011" rpy="${pi} 0 0"/>
+        <mass value="${proximal_link_mass}"/>
+        <xacro:cuboid_inertia m="${proximal_link_mass}" x="0.02" y="0.15" z="0.071"/>
+      </inertial>
+      <collision>
+        <origin xyz="-0.011 0.007 0.011" rpy="${pi} 0 0"/>
+        <geometry>
+          <mesh filename="${mesh_path}/proximal_coll.STL"/>
+        </geometry>
       </collision>
     </link>
@@ -76,20 +86,20 @@
     <link name="distal_${finger_id}">
       <visual>
-	<origin xyz="-0.077 0.007 0.007" rpy="${pi} 0 0"/>
-	<geometry>
+        <origin xyz="-0.077 0.007 0.007" rpy="${pi} 0 0"/>
+        <geometry>
           <mesh filename="${mesh_path}/distal.STL"/>
-	</geometry>
-	<material name="black"/>
-      </visual>
-      <inertial>
-	<origin xyz="-0.077 0.007 0.007" rpy="3.1459 0 0"/>
-	<mass value="${distal_link_mass}"/>
-	<xacro:cuboid_inertia m="${distal_link_mass}" x="0.017" y="0.15" z="0.039"/>
-      </inertial>
-      <collision>
-	<origin xyz="-0.077 0.007 0.007" rpy="${pi} 0 0"/>
-	<geometry>
-	  <mesh filename="${mesh_path}/distal_coll.STL"/>
-	</geometry>
+        </geometry>
+        <material name="black"/>
+      </visual>
+      <inertial>
+        <origin xyz="-0.077 0.007 0.007" rpy="3.1459 0 0"/>
+        <mass value="${distal_link_mass}"/>
+        <xacro:cuboid_inertia m="${distal_link_mass}" x="0.017" y="0.15" z="0.039"/>
+      </inertial>
+      <collision>
+        <origin xyz="-0.077 0.007 0.007" rpy="${pi} 0 0"/>
+        <geometry>
+          <mesh filename="${mesh_path}/distal_coll.STL"/>
+        </geometry>
       </collision>
     </link>
@@ -98,22 +108,20 @@
     <link name="proximal_${finger_id}_pad">
       <visual>
-	<origin xyz="-0.008 0.014 -0.002" rpy="${pi/2} ${pi/2} 0" />
-	<geometry>
+        <origin xyz="-0.008 0.014 -0.002" rpy="${pi/2} ${pi/2} 0" />
+        <geometry>
           <mesh filename="${mesh_path}/proximal_pad.STL"/>
-	</geometry>
-	<material name="dark_grey">
-	  <color rgba="0.2 0.2 0.2 1"/>
-	</material>
-      </visual>
-      <inertial>
-	<origin xyz="-0.008 0.014 -0.002" rpy="${pi/2} ${pi/2} 0"/>
-	<mass value="${proximal_pad_mass}"/>
-	<xacro:cuboid_inertia m="${proximal_pad_mass}" x="0.005" y="0.15" z="0.071"/>
-      </inertial>
-      <collision>
-	<origin xyz="-0.008 0.014 -0.002" rpy="${pi/2} ${pi/2} 0"/>
-	<geometry>
-	  <mesh filename="${mesh_path}/proximal_pad_coll.STL"/>
-	</geometry>
+        </geometry>
+        <material name="dark_grey"/>
+      </visual>
+      <inertial>
+        <origin xyz="-0.008 0.014 -0.002" rpy="${pi/2} ${pi/2} 0"/>
+        <mass value="${proximal_pad_mass}"/>
+        <xacro:cuboid_inertia m="${proximal_pad_mass}" x="0.005" y="0.15" z="0.071"/>
+      </inertial>
+      <collision>
+        <origin xyz="-0.008 0.014 -0.002" rpy="${pi/2} ${pi/2} 0"/>
+        <geometry>
+          <mesh filename="${mesh_path}/proximal_pad_coll.STL"/>
+        </geometry>
       </collision>
     </link>
@@ -122,22 +130,20 @@
     <link name="distal_${finger_id}_pad">
       <visual>
-	<origin xyz="-0.00825 0.009 0.057" rpy="${pi/2} ${pi/2} 0"/>
-	<geometry>
+        <origin xyz="-0.00825 0.009 0.057" rpy="${pi/2} ${pi/2} 0"/>
+        <geometry>
           <mesh filename="${mesh_path}/distal_pad.STL"/>
-	</geometry>
-	<material name="dark_grey">
-	  <color rgba="0.2 0.2 0.2 1"/>
-	</material>
-      </visual>
-      <inertial>
-	<origin xyz="-0.00825 0.009 0.057" rpy="${pi/2} ${pi/2} 0"/>
-	<mass value="${distal_pad_mass}"/>
-	<xacro:cuboid_inertia m="${distal_pad_mass}" x="0.005" y="0.15" z="0.039"/>
-      </inertial>
-      <collision>
-	<origin xyz="-0.00825 0.009 0.057" rpy="${pi/2} ${pi/2} 0"/>
-	<geometry>
-	  <mesh filename="${mesh_path}/distal_pad_coll.STL"/>
-	</geometry>
+        </geometry>
+        <material name="dark_grey"/>
+      </visual>
+      <inertial>
+        <origin xyz="-0.00825 0.009 0.057" rpy="${pi/2} ${pi/2} 0"/>
+        <mass value="${distal_pad_mass}"/>
+        <xacro:cuboid_inertia m="${distal_pad_mass}" x="0.005" y="0.15" z="0.039"/>
+      </inertial>
+      <collision>
+        <origin xyz="-0.00825 0.009 0.057" rpy="${pi/2} ${pi/2} 0"/>
+        <geometry>
+          <mesh filename="${mesh_path}/distal_pad_coll.STL"/>
+        </geometry>
       </collision>
     </link>
@@ -146,20 +152,20 @@
     <link name="swivel_${finger_id}">
       <visual>
-	<origin xyz="0 0 0" rpy="0 0 0"/>
-	<geometry>
+        <origin xyz="0 0 0" rpy="0 0 0"/>
+        <geometry>
           <mesh filename="${mesh_path}/swivel_${finger_id}.STL"/>
-	</geometry>
-	<material name="black"/>
-      </visual>
-      <inertial>
-	<origin xyz="0 0 0" rpy="0 0 0"/>
-	<mass value="${swivel_link_mass}"/>
-	<xacro:cuboid_inertia m="${swivel_link_mass}" x="0.022" y="0.032" z="0.03"/>
-      </inertial>
-      <collision>
-	<origin xyz="0 0 0" rpy="0 0 0"/>
-	<geometry>
-	  <mesh filename="${mesh_path}/swivel_${finger_id}_coll.STL"/>
-	</geometry>
+        </geometry>
+        <material name="black"/>
+      </visual>
+      <inertial>
+        <origin xyz="0 0 0" rpy="0 0 0"/>
+        <mass value="${swivel_link_mass}"/>
+        <xacro:cuboid_inertia m="${swivel_link_mass}" x="0.022" y="0.032" z="0.03"/>
+      </inertial>
+      <collision>
+        <origin xyz="0 0 0" rpy="0 0 0"/>
+        <geometry>
+          <mesh filename="${mesh_path}/swivel_${finger_id}_coll.STL"/>
+        </geometry>
       </collision>
     </link>
@@ -168,20 +174,20 @@
     <link name="shell">
       <visual>
-	<origin xyz="0 0 0" rpy="0 0 0"/>
-	<geometry>
+        <origin xyz="0 0 0" rpy="0 0 0"/>
+        <geometry>
           <mesh filename="${mesh_path}/base_link.STL"/>
-	</geometry>
-	<material name="black"/>
-      </visual>
-      <inertial>
-	<origin xyz="0 0 0" rpy="0 0 0"/>
-	<mass value="${shell_mass}"/>
-	<xacro:cuboid_inertia m="${shell_mass}" x="0.066" y="0.091" z="0.136"/>
-      </inertial>
-      <collision>
-	<origin xyz="0 0 0" rpy="0 0 0"/>
-	<geometry>
-	  <mesh filename="${mesh_path}/base_link_coll.STL"/>
-	</geometry>
+        </geometry>
+        <material name="black"/>
+      </visual>
+      <inertial>
+        <origin xyz="0 0 0" rpy="0 0 0"/>
+        <mass value="${shell_mass}"/>
+        <xacro:cuboid_inertia m="${shell_mass}" x="0.066" y="0.091" z="0.136"/>
+      </inertial>
+      <collision>
+        <origin xyz="0 0 0" rpy="0 0 0"/>
+        <geometry>
+          <mesh filename="${mesh_path}/base_link_coll.STL"/>
+        </geometry>
       </collision>
     </link>
@@ -190,26 +196,24 @@
     <link name="pad">
       <visual>
-	<origin xyz="0 0 0" rpy="0 0 0"/>
-	<geometry>
+        <origin xyz="0 0 0" rpy="0 0 0"/>
+        <geometry>
           <mesh filename="${mesh_path}/pad.STL"/>
-	</geometry>
-	<material name="dark_grey">
-	  <color rgba="0.2 0.2 0.2 1"/>
-	</material>
-      </visual>
-      <inertial>
-	<origin xyz="0 0 0" rpy="0 0 0"/>
-	<mass value="${pad_mass}"/>
-	<xacro:cuboid_inertia m="${pad_mass}" x="0.066" y="0.091" z="0.136"/>
-      </inertial>
-      <collision>
-	<origin xyz="0 0 0" rpy="0 0 0"/>
-	<geometry>
-	  <mesh filename="${mesh_path}/pad_coll.STL"/>
-	</geometry>
-      </collision>
-    </link>
-  </xacro:macro>
-  <link name="palm_link" /> <!-- A dummy link to define the end-effector frame -->
+        </geometry>
+        <material name="dark_grey"/>
+      </visual>
+      <inertial>
+        <origin xyz="0 0 0" rpy="0 0 0"/>
+        <mass value="${pad_mass}"/>
+        <xacro:cuboid_inertia m="${pad_mass}" x="0.066" y="0.091" z="0.136"/>
+      </inertial>
+      <collision>
+        <origin xyz="0 0 0" rpy="0 0 0"/>
+        <geometry>
+          <mesh filename="${mesh_path}/pad_coll.STL"/>
+        </geometry>
+      </collision>
+    </link>
+  </xacro:macro>
+  <link name="palm_link" />
   <!-- =================================== Tactile macros =================================== -->
   <!-- Sensor links are rendered only to give a link that the Gazebo sensor plugin can latch  -->
@@ -221,19 +225,19 @@
     <link name="${location}_${finger_id}_sensor_${sensor_id}">
       <visual>
-      	<origin xyz="0 0 0" rpy="0 0 0"/>
-      	<geometry>
-      	  <box size="0.006 0.006 0.0003"/>
-      	</geometry>
-      </visual>
-      <inertial>
-	<origin xyz="0 0 0" rpy="0 0 0"/>
-	<mass value="1e-5"/>
-	<xacro:cuboid_inertia m="1e-5" x="0.006" y="0.006" z="0.0003"/>
-      </inertial>
-      <collision>
-      	<origin xyz="0 0 0" rpy="0 0 0"/>
-      	<geometry>
-      	  <box size="0.006 0.006 0.0003"/>
-      	</geometry>
+        <origin xyz="0 0 0" rpy="0 0 0"/>
+        <geometry>
+          <box size="0.006 0.006 0.0003"/>
+        </geometry>
+      </visual>
+      <inertial>
+        <origin xyz="0 0 0" rpy="0 0 0"/>
+        <mass value="1e-5"/>
+        <xacro:cuboid_inertia m="1e-5" x="0.006" y="0.006" z="0.0003"/>
+      </inertial>
+      <collision>
+        <origin xyz="0 0 0" rpy="0 0 0"/>
+        <geometry>
+          <box size="0.006 0.006 0.0003"/>
+        </geometry>
       </collision>
     </link>
@@ -242,12 +246,12 @@
     <joint name="${location}_${finger_id}_to_sensor_${sensor_id}" type="fixed">
       <xacro:if value="${location == 'proximal'}">
-	<xacro:property name="x_offset" value="0.012"/>
-	<xacro:property name="x_gap"    value="0.008"/>
-	<xacro:property name="z_offset" value="0.014"/>
+        <xacro:property name="x_offset" value="0.012"/>
+        <xacro:property name="x_gap" value="0.008"/>
+        <xacro:property name="z_offset" value="0.014"/>
       </xacro:if>
       <xacro:if value="${location == 'distal'}">
-	<xacro:property name="x_offset" value="0.008"/>
-	<xacro:property name="x_gap"    value="0.008"/>
-	<xacro:property name="z_offset" value="0.01"/>
+        <xacro:property name="x_offset" value="0.008"/>
+        <xacro:property name="x_gap" value="0.008"/>
+        <xacro:property name="z_offset" value="0.01"/>
       </xacro:if>
       <origin xyz="${x_offset + x_gap * sensor_id} 0 ${z_offset}" rpy="0 0 0"/>
@@ -306,10 +310,10 @@
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