Commit message: Integrate Gazebo ROS Bumper plugin

File: description/urdf/reflex/reflex.gazebo.xacro (robot description, xacro)
@@ -2,7 +2,5 @@
 <robot xmlns:xacro="http://www.ros.org/wiki/xacro">
   <!-- ============================== Transmissions ============================== -->
-  <xacro:if value="$(arg actuate_reflex)">
-    <xacro:include filename="$(find description)/urdf/reflex/reflex.transmission.xacro"/>
-  </xacro:if>
+  <xacro:include filename="$(find description)/urdf/reflex/reflex.transmission.xacro"/>
   <!-- ================================ Materials ================================ -->
   <xacro:macro name="color_swivel" params="finger_id">
@@ -36,16 +34,27 @@
     </gazebo>
   </xacro:macro>
-  <!-- ========================== Contact/Pressure sensors =========================== -->
-  <xacro:macro name="reflex_sensor" params="type location finger_id sensor_id">
-    <gazebo reference="${location}_${finger_id}_sensor_${sensor_id}">
-      <xacro:property name="sensor_name"
-		      value="reflex/${location}_${finger_id}_${type}_sensor_${sensor_id}"/>
+  <gazebo reference="shell">
+    <material>Gazebo/Black</material>
+  </gazebo>
+  <gazebo reference="pad">
+    <material>Gazebo/FlatBlack</material>
+  </gazebo>
+  <!-- ========================== Contact Sensors =========================== -->
+  <xacro:macro name="reflex_sensor" params="location finger_id sensor_id">
+    <xacro:property name="link_name" value="${location}_${finger_id}_sensor_${sensor_id}"/>
+    <xacro:property name="sensor_name" value="reflex/${link_name}"/>
+    <gazebo reference="${link_name}">
+      <selfCollide value="true" />
       <sensor name="${sensor_name}" type="contact">
-	<plugin name="${sensor_name}_plugin" filename="lib${type}_sensor_plugin.so">
-	  <updateRate>100</updateRate> <!-- In range [0, 1000] -->
-	</plugin>
-	<contact>
-	  <collision>${sensor_name}_collision</collision> <!-- Auto-determined by SDF -->
-	</contact>
+        <alwaysOn>true</alwaysOn>
+        <!-- 50 Hz is the real sampling rate of the Reflex tactile sensors -->
+        <update_rate>50</update_rate>
+        <plugin name="${sensor_name}_plugin" filename="libgazebo_ros_bumper.so">
+          <bumperTopicName>${sensor_name}_bumper</bumperTopicName>
+          <frameName>${link_name}</frameName>
+        </plugin>
+        <contact>
+          <collision>${link_name}_collision</collision>
+        </contact>
       </sensor>
       <material>Gazebo/GreenTransparent</material>
@@ -57,20 +66,20 @@
     </gazebo>
   </xacro:macro>
-  <xacro:macro name="gazebo_finger" params="sensor_type id">
-    <xacro:color_swivel       finger_id="${id}"/>
-    <xacro:color_distal       finger_id="${id}"/>
-    <xacro:color_proximal     finger_id="${id}"/>
-    <xacro:color_distal_pad   finger_id="${id}"/>
+  <xacro:macro name="gazebo_finger" params="id">
+    <xacro:color_swivel finger_id="${id}"/>
+    <xacro:color_distal finger_id="${id}"/>
+    <xacro:color_proximal finger_id="${id}"/>
+    <xacro:color_distal_pad finger_id="${id}"/>
     <xacro:color_proximal_pad finger_id="${id}"/>
-    <xacro:color_flex         finger_id="${id}"/>
-    <xacro:reflex_sensor type="${sensor_type}" location="proximal" finger_id="${id}" sensor_id="1"/>
-    <xacro:reflex_sensor type="${sensor_type}" location="proximal" finger_id="${id}" sensor_id="2"/>
-    <xacro:reflex_sensor type="${sensor_type}" location="proximal" finger_id="${id}" sensor_id="3"/>
-    <xacro:reflex_sensor type="${sensor_type}" location="proximal" finger_id="${id}" sensor_id="4"/>
-    <xacro:reflex_sensor type="${sensor_type}" location="proximal" finger_id="${id}" sensor_id="5"/>
-    <xacro:reflex_sensor type="${sensor_type}" location="distal"   finger_id="${id}" sensor_id="1"/>
-    <xacro:reflex_sensor type="${sensor_type}" location="distal"   finger_id="${id}" sensor_id="2"/>
-    <xacro:reflex_sensor type="${sensor_type}" location="distal"   finger_id="${id}" sensor_id="3"/>
-    <xacro:reflex_sensor type="${sensor_type}" location="distal"   finger_id="${id}" sensor_id="4"/>
+    <xacro:color_flex finger_id="${id}"/>
+    <xacro:reflex_sensor location="proximal" finger_id="${id}" sensor_id="1"/>
+    <xacro:reflex_sensor location="proximal" finger_id="${id}" sensor_id="2"/>
+    <xacro:reflex_sensor location="proximal" finger_id="${id}" sensor_id="3"/>
+    <xacro:reflex_sensor location="proximal" finger_id="${id}" sensor_id="4"/>
+    <xacro:reflex_sensor location="proximal" finger_id="${id}" sensor_id="5"/>
+    <xacro:reflex_sensor location="distal" finger_id="${id}" sensor_id="1"/>
+    <xacro:reflex_sensor location="distal" finger_id="${id}" sensor_id="2"/>
+    <xacro:reflex_sensor location="distal" finger_id="${id}" sensor_id="3"/>
+    <xacro:reflex_sensor location="distal" finger_id="${id}" sensor_id="4"/>
     <xacro:preserve_fixed location="proximal" finger_id="${id}" sensor_id="1"/>
     <xacro:preserve_fixed location="proximal" finger_id="${id}" sensor_id="2"/>
@@ -78,20 +87,11 @@
     <xacro:preserve_fixed location="proximal" finger_id="${id}" sensor_id="4"/>
     <xacro:preserve_fixed location="proximal" finger_id="${id}" sensor_id="5"/>
-    <xacro:preserve_fixed location="distal"   finger_id="${id}" sensor_id="1"/>
-    <xacro:preserve_fixed location="distal"   finger_id="${id}" sensor_id="2"/>
-    <xacro:preserve_fixed location="distal"   finger_id="${id}" sensor_id="3"/>
-    <xacro:preserve_fixed location="distal"   finger_id="${id}" sensor_id="4"/>
+    <xacro:preserve_fixed location="distal" finger_id="${id}" sensor_id="1"/>
+    <xacro:preserve_fixed location="distal" finger_id="${id}" sensor_id="2"/>
+    <xacro:preserve_fixed location="distal" finger_id="${id}" sensor_id="3"/>
+    <xacro:preserve_fixed location="distal" finger_id="${id}" sensor_id="4"/>
   </xacro:macro>
-  <!-- ================================================================================ -->
-  <!-- These use the preceding macros to set colors and add sensors to the fingers -->
-  <gazebo reference="shell">
-    <material>Gazebo/Black</material>
-  </gazebo>
-  <gazebo reference="pad">
-    <material>Gazebo/FlatBlack</material>
-  </gazebo>
-  <!-- TODO create an arg for sensor type when done testing -->
-  <xacro:gazebo_finger sensor_type="pressure" id="1"/>
-  <xacro:gazebo_finger sensor_type="pressure" id="2"/>
-  <xacro:gazebo_finger sensor_type="pressure" id="3"/>
+  <xacro:gazebo_finger id="1"/>
+  <xacro:gazebo_finger id="2"/>
+  <xacro:gazebo_finger id="3"/>
 </robot>

Commit message: Change sensor namespace from "reflex" to "gazebo"

File: description/urdf/reflex/reflex.gazebo.xacro (robot description, xacro)
@@ -56,5 +56,5 @@
   <xacro:macro name="reflex_sensor" params="location finger_id sensor_id">
     <xacro:property name="link_name" value="${location}_${finger_id}_sensor_${sensor_id}"/>
-    <xacro:property name="sensor_name" value="reflex/${link_name}"/>
+    <xacro:property name="sensor_name" value="gazebo/${link_name}"/>
     <gazebo reference="${link_name}">
       <selfCollide value="true" />
