Commit message: Add PID position controllers for flexure

File: simulation/description/urdf/reflex/reflex.transmission.xacro (robot description, xacro)
@@ -1,32 +1,62 @@
 <?xml version="1.0"?>
 <robot xmlns:xacro="http://www.ros.org/wiki/xacro">
-  <xacro:macro name="reflex_preshape_transmission" params="finger_id">
+  <xacro:macro name="preshape_transmission" params="finger_id">
     <transmission name="preshape_${finger_id}_transmission">
       <type>transmission_interface/SimpleTransmission</type>
       <joint name="preshape_${finger_id}">
-	<hardwareInterface>hardware_interface/EffortJointInterface</hardwareInterface>
+        <hardwareInterface>hardware_interface/EffortJointInterface</hardwareInterface>
       </joint>
       <actuator name="preshape_${finger_id}_motor">
-	<hardwareInterface>hardware_interface/EffortJointInterface</hardwareInterface>
-	<mechanicalReduction>1</mechanicalReduction>
+        <hardwareInterface>hardware_interface/EffortJointInterface</hardwareInterface>
+        <mechanicalReduction>1</mechanicalReduction>
       </actuator>
     </transmission>
   </xacro:macro>
-  <xacro:macro name="reflex_proximal_joint_transmission" params="finger_id">
+  <xacro:macro name="proximal_joint_transmission" params="finger_id">
     <transmission name="proximal_joint_${finger_id}_transmission">
       <type>transmission_interface/SimpleTransmission</type>
       <joint name="proximal_joint_${finger_id}">
-	<hardwareInterface>hardware_interface/EffortJointInterface</hardwareInterface>
+        <hardwareInterface>hardware_interface/EffortJointInterface</hardwareInterface>
       </joint>
       <actuator name="proximal_joint_${finger_id}_motor">
-	<hardwareInterface>hardware_interface/EffortJointInterface</hardwareInterface>
-	<mechanicalReduction>1</mechanicalReduction>
+        <hardwareInterface>hardware_interface/EffortJointInterface</hardwareInterface>
+        <mechanicalReduction>1</mechanicalReduction>
       </actuator>
     </transmission>
   </xacro:macro>
-  <xacro:reflex_preshape_transmission finger_id="1"/>
-  <xacro:reflex_preshape_transmission finger_id="2"/>
-  <xacro:reflex_proximal_joint_transmission finger_id="1"/>
-  <xacro:reflex_proximal_joint_transmission finger_id="2"/>
-  <xacro:reflex_proximal_joint_transmission finger_id="3"/>
+  <xacro:macro name="proximal_to_flex_joint_transmission" params="finger_id">
+    <transmission name="proximal_to_flex_joint_${finger_id}_transmission">
+      <type>transmission_interface/SimpleTransmission</type>
+      <joint name="proximal_${finger_id}_to_flex">
+        <hardwareInterface>hardware_interface/EffortJointInterface</hardwareInterface>
+      </joint>
+      <actuator name="proximal_${finger_id}_to_flex_motor">
+        <hardwareInterface>hardware_interface/EffortJointInterface</hardwareInterface>
+        <mechanicalReduction>1</mechanicalReduction>
+      </actuator>
+    </transmission>
+  </xacro:macro>
+  <xacro:macro name="flex_to_distal_joint_transmission" params="finger_id">
+    <transmission name="flex_to_distal_${finger_id}_transmission">
+      <type>transmission_interface/SimpleTransmission</type>
+      <joint name="flex_to_distal_${finger_id}">
+        <hardwareInterface>hardware_interface/EffortJointInterface</hardwareInterface>
+      </joint>
+      <actuator name="flex_to_distal_${finger_id}_motor">
+        <hardwareInterface>hardware_interface/EffortJointInterface</hardwareInterface>
+        <mechanicalReduction>1</mechanicalReduction>
+      </actuator>
+    </transmission>
+  </xacro:macro>
+  <xacro:preshape_transmission finger_id="1"/>
+  <xacro:preshape_transmission finger_id="2"/>
+  <xacro:proximal_joint_transmission finger_id="1"/>
+  <xacro:proximal_joint_transmission finger_id="2"/>
+  <xacro:proximal_joint_transmission finger_id="3"/>
+  <xacro:proximal_to_flex_joint_transmission finger_id="1"/>
+  <xacro:proximal_to_flex_joint_transmission finger_id="2"/>
+  <xacro:proximal_to_flex_joint_transmission finger_id="3"/>
+  <xacro:flex_to_distal_joint_transmission finger_id="1"/>
+  <xacro:flex_to_distal_joint_transmission finger_id="2"/>
+  <xacro:flex_to_distal_joint_transmission finger_id="3"/>
 </robot>
