Commit message: Add debug node for forces and penetration depths

File: simulation/description/urdf/reflex/reflex.gazebo.xacro (robot description, xacro)
@@ -54,5 +54,6 @@
   </gazebo>
   <!-- ========================== Contact Sensors =========================== -->
-  <xacro:macro name="reflex_sensor" params="location finger_id sensor_id">
+  <!-- adds sensor plugin to sensor links -->
+  <xacro:macro name="tactile_sensor" params="location finger_id sensor_id">
     <xacro:property name="link_name" value="${location}_${finger_id}_sensor_${sensor_id}"/>
     <xacro:property name="sensor_name" value="gazebo/${link_name}"/>
@@ -73,4 +74,22 @@
     </gazebo>
   </xacro:macro>
+  <!-- adds sensor plugin to proximal and distal links -->
+  <xacro:macro name="link_sensor" params="location finger_id">
+    <xacro:property name="link_name" value="${location}_${finger_id}"/>
+    <xacro:property name="sensor_name" value="gazebo/${link_name}_sensor"/>
+    <gazebo reference="${link_name}">
+      <sensor name="${sensor_name}" type="contact">
+        <alwaysOn>true</alwaysOn>
+        <update_rate>50</update_rate>
+        <plugin name="${sensor_name}_plugin" filename="libgazebo_ros_bumper.so">
+          <bumperTopicName>${sensor_name}_bumper</bumperTopicName>
+          <frameName>${link_name}</frameName>
+        </plugin>
+        <contact>
+          <collision>${link_name}_collision</collision>
+        </contact>
+      </sensor>
+    </gazebo>
+  </xacro:macro>
   <xacro:macro name="preserve_fixed" params="location finger_id sensor_id">
     <gazebo reference="${location}_${finger_id}_to_sensor_${sensor_id}">
@@ -85,13 +104,15 @@
     <xacro:color_proximal_pad finger_id="${id}"/>
     <xacro:color_flex finger_id="${id}"/>
-    <xacro:reflex_sensor location="proximal" finger_id="${id}" sensor_id="1"/>
-    <xacro:reflex_sensor location="proximal" finger_id="${id}" sensor_id="2"/>
-    <xacro:reflex_sensor location="proximal" finger_id="${id}" sensor_id="3"/>
-    <xacro:reflex_sensor location="proximal" finger_id="${id}" sensor_id="4"/>
-    <xacro:reflex_sensor location="proximal" finger_id="${id}" sensor_id="5"/>
-    <xacro:reflex_sensor location="distal" finger_id="${id}" sensor_id="1"/>
-    <xacro:reflex_sensor location="distal" finger_id="${id}" sensor_id="2"/>
-    <xacro:reflex_sensor location="distal" finger_id="${id}" sensor_id="3"/>
-    <xacro:reflex_sensor location="distal" finger_id="${id}" sensor_id="4"/>
+    <xacro:tactile_sensor location="proximal" finger_id="${id}" sensor_id="1"/>
+    <xacro:tactile_sensor location="proximal" finger_id="${id}" sensor_id="2"/>
+    <xacro:tactile_sensor location="proximal" finger_id="${id}" sensor_id="3"/>
+    <xacro:tactile_sensor location="proximal" finger_id="${id}" sensor_id="4"/>
+    <xacro:tactile_sensor location="proximal" finger_id="${id}" sensor_id="5"/>
+    <xacro:tactile_sensor location="distal" finger_id="${id}" sensor_id="1"/>
+    <xacro:tactile_sensor location="distal" finger_id="${id}" sensor_id="2"/>
+    <xacro:tactile_sensor location="distal" finger_id="${id}" sensor_id="3"/>
+    <xacro:tactile_sensor location="distal" finger_id="${id}" sensor_id="4"/>
+    <xacro:link_sensor location="proximal" finger_id="${id}"/>
+    <xacro:link_sensor location="distal" finger_id="${id}"/>
     <xacro:preserve_fixed location="proximal" finger_id="${id}" sensor_id="1"/>
     <xacro:preserve_fixed location="proximal" finger_id="${id}" sensor_id="2"/>
