Commit message: Change joint velocity limits

File: simulation/description/urdf/reflex/reflex.urdf.xacro (robot description, xacro)
@@ -309,5 +309,5 @@
       <child link="swivel_${finger_id}"/>
       <dynamics damping="0.1" />
-      <limit effort="15" lower="0.0" upper="${pi/2}" velocity="7"/>
+      <limit effort="0.2" lower="0.0" upper="${pi/2}" velocity="0.01"/>
       <xacro:if value="${finger_id == 1}">
         <origin xyz="0.0503973683071414 -0.026 0.063" rpy="0 0 0"/>
@@ -325,5 +325,5 @@
       <axis xyz="0 -1 0"/>
       <dynamics damping="0.1" />
-      <limit effort="15" lower="0.0" upper="${pi}" velocity="7"/>
+      <limit effort="0.2" lower="0.0" upper="${pi}" velocity="0.01"/>
       <xacro:if value="${finger_id == 3}">
         <origin xyz="-0.03 0 0.0816" rpy="0 0.28 ${pi}"/>

Commit message: Improve inertia values

File: simulation/description/urdf/reflex/reflex.urdf.xacro (robot description, xacro)
@@ -26,39 +26,46 @@
   </material>
   <!-- ======================================= Masses ======================================== -->
-  <!-- These are rough approximations, the total hand mass was measured to be about 0.9kg,     -->
-  <!-- most of it concentrated in the shell anyways, so for sake of arm controller, most mass  -->
-  <!-- is being given to shell/pad, treating fingers as almost massless, so that KDL chain for -->
-  <!-- arm can just go through the palm pad and be accounting for most of the hand mass.       -->
+  <!-- These are rough approximations, the total hand mass was measured to be about 0.9kg     -->
+  <!-- final mass: 0.6+0.03+2*0.02+3*(0.025+0.015+0.01+0.02+0.01) = 0.91 -->
+  <xacro:property name="shell_mass" value="0.6"/>
+  <xacro:property name="pad_mass" value="0.03"/>
+  <!-- these links occur twice -->
+  <xacro:property name="swivel_link_mass" value="0.02"/>
+  <!-- these links occur three times (once on each finger) -->
+  <xacro:property name="proximal_link_mass" value="0.025"/>
+  <xacro:property name="proximal_pad_mass" value="0.015"/>
   <xacro:property name="flex_link_mass" value="0.01"/>
-  <xacro:property name="proximal_link_mass" value="0.01"/>
-  <xacro:property name="distal_link_mass" value="0.01"/>
-  <xacro:property name="proximal_pad_mass" value="0.01"/>
+  <xacro:property name="distal_link_mass" value="0.02"/>
   <xacro:property name="distal_pad_mass" value="0.01"/>
-  <xacro:property name="swivel_link_mass" value="0.01"/>
-  <xacro:property name="shell_mass" value="0.74"/>
-  <xacro:property name="pad_mass" value="0.1"/>
   <!-- ====================================== Link Macros ==================================== -->
+  <xacro:property name="flex_link_box_x" value="0.017"/>
+  <xacro:property name="flex_link_box_y" value="0.014"/>
+  <xacro:property name="flex_link_box_z" value="0.0065"/>
   <xacro:macro name="flex_link" params="finger_id">
     <link name="finger_${finger_id}_flex_link">
       <visual>
-        <origin xyz="0.0005 0 -0.003" rpy="0 0 0"/>
-        <geometry>
-          <box size="0.017 0.014 0.0065"/>
+        <origin xyz="${flex_link_box_x/2} 0 ${flex_link_box_z/2}" rpy="0 0 0"/>
+        <geometry>
+          <box size="${flex_link_box_x} ${flex_link_box_y} ${flex_link_box_z}"/>
         </geometry>
         <material name="gold"/>
       </visual>
       <inertial>
-        <origin xyz="0 0 0" rpy="0 0 0"/>
+        <origin xyz="${flex_link_box_x/2} 0 ${flex_link_box_z/2}" rpy="0 0 0"/>
         <mass value="${flex_link_mass}"/>
-        <xacro:cuboid_inertia m="${flex_link_mass}" x="0.005" y="0.014" z="0.015"/>
-      </inertial>
-      <collision>
-        <origin xyz="0 0 0" rpy="0 0 0"/>
-        <geometry>
-          <box size="0.01 0.01 0.01"/>
-        </geometry>
-      </collision>
-    </link>
-  </xacro:macro>
+        <xacro:cuboid_inertia m="${flex_link_mass}" x="${flex_link_box_x}" y="${flex_link_box_y}" z="${flex_link_box_z}"/>
+      </inertial>
+      <collision>
+        <origin xyz="${flex_link_box_x/2} 0 ${flex_link_box_z/2}" rpy="0 0 0"/>
+        <geometry>
+          <box size="${flex_link_box_x} ${flex_link_box_y} ${flex_link_box_z}"/>
+        </geometry>
+      </collision>
+    </link>
+  </xacro:macro>
+  <!-- approx length, height and width of a cuboid surrounding the link -->
+  <xacro:property name="proximal_link_box_x" value="0.071"/>
+  <xacro:property name="proximal_link_box_y" value="0.014"/>
+  <xacro:property name="proximal_link_box_z" value="0.012"/>
   <xacro:macro name="proximal_link" params="finger_id">
     <link name="proximal_${finger_id}">
@@ -71,10 +78,10 @@
       </visual>
       <inertial>
+        <origin xyz="${proximal_link_box_x/2-0.011} 0 0" rpy="0 0 0"/>
+        <mass value="${proximal_link_mass}"/>
+        <xacro:cuboid_inertia m="${proximal_link_mass}" x="${proximal_link_box_x}" y="${proximal_link_box_y}" z="${proximal_link_box_z}"/>
+      </inertial>
+      <collision>
         <origin xyz="-0.011 0.007 0.011" rpy="${pi} 0 0"/>
-        <mass value="${proximal_link_mass}"/>
-        <xacro:cuboid_inertia m="${proximal_link_mass}" x="0.02" y="0.15" z="0.071"/>
-      </inertial>
-      <collision>
-        <origin xyz="-0.011 0.007 0.011" rpy="${pi} 0 0"/>
         <geometry>
           <mesh filename="${mesh_path}/proximal_coll.STL"/>
@@ -83,8 +90,12 @@
     </link>
   </xacro:macro>
+  <!-- approx length, height and width of a cuboid surrounding the link -->
+  <xacro:property name="distal_link_box_x" value="0.036"/>
+  <xacro:property name="distal_link_box_y" value="${proximal_link_box_y}"/>
+  <xacro:property name="distal_link_box_z" value="0.012"/>
   <xacro:macro name="distal_link" params="finger_id">
     <link name="distal_${finger_id}">
       <visual>
-        <origin xyz="-0.077 0.007 0.007" rpy="${pi} 0 0"/>
+        <origin xyz="${-0.077-flex_link_box_x/2} 0.007 ${0.007+flex_link_box_z/2+0.004+flex_z_offset}" rpy="${pi} 0 0"/>
         <geometry>
           <mesh filename="${mesh_path}/distal.STL"/>
@@ -93,10 +104,10 @@
       </visual>
       <inertial>
-        <origin xyz="-0.077 0.007 0.007" rpy="3.1459 0 0"/>
+        <origin xyz="${distal_link_box_x/2} 0 ${distal_link_box_z/2-0.002}" rpy="0 0 0"/>
         <mass value="${distal_link_mass}"/>
-        <xacro:cuboid_inertia m="${distal_link_mass}" x="0.017" y="0.15" z="0.039"/>
-      </inertial>
-      <collision>
-        <origin xyz="-0.077 0.007 0.007" rpy="${pi} 0 0"/>
+        <xacro:cuboid_inertia m="${distal_link_mass}" x="${distal_link_box_x}" y="${distal_link_box_y}" z="${distal_link_box_z}"/>
+      </inertial>
+      <collision>
+        <origin xyz="${-0.077-flex_link_box_x/2} 0.007 ${0.007+flex_link_box_z/2}" rpy="${pi} 0 0"/>
         <geometry>
           <mesh filename="${mesh_path}/distal_coll.STL"/>
@@ -105,4 +116,7 @@
     </link>
   </xacro:macro>
+  <xacro:property name="proximal_pad_box_x" value="0.016"/>
+  <xacro:property name="proximal_pad_box_y" value="0.020"/>
+  <xacro:property name="proximal_pad_box_z" value="0.05"/>
   <xacro:macro name="proximal_pad" params="finger_id">
     <link name="proximal_${finger_id}_pad">
@@ -115,10 +129,10 @@
       </visual>
       <inertial>
+        <origin xyz="0 0.004 -0.035" rpy="0 0 0"/>
+        <mass value="${proximal_pad_mass}"/>
+        <xacro:cuboid_inertia m="${proximal_pad_mass}" x="${proximal_pad_box_x}" y="${proximal_pad_box_y}" z="${proximal_pad_box_z}"/>
+      </inertial>
+      <collision>
         <origin xyz="-0.008 0.014 -0.002" rpy="${pi/2} ${pi/2} 0"/>
-        <mass value="${proximal_pad_mass}"/>
-        <xacro:cuboid_inertia m="${proximal_pad_mass}" x="0.005" y="0.15" z="0.071"/>
-      </inertial>
-      <collision>
-        <origin xyz="-0.008 0.014 -0.002" rpy="${pi/2} ${pi/2} 0"/>
         <geometry>
           <mesh filename="${mesh_path}/proximal_pad_coll.STL"/>
@@ -127,8 +141,12 @@
     </link>
   </xacro:macro>
+  <xacro:property name="distal_pad_box_x" value="${proximal_pad_box_x}"/>
+  <xacro:property name="distal_pad_box_y" value="0.018"/>
+  <xacro:property name="distal_pad_box_z" value="0.037"/>
   <xacro:macro name="distal_pad" params="finger_id">
     <link name="distal_${finger_id}_pad">
       <visual>
-        <origin xyz="-0.00825 0.009 0.057" rpy="${pi/2} ${pi/2} 0"/>
+        <!-- setting these xyz values by eye as transformations get too complex -->
+        <origin xyz="-0.008 0.0155 0.076" rpy="${pi/2} ${pi/2} 0"/>
         <geometry>
           <mesh filename="${mesh_path}/distal_pad.STL"/>
@@ -137,10 +155,10 @@
       </visual>
       <inertial>
-        <origin xyz="-0.00825 0.009 0.057" rpy="${pi/2} ${pi/2} 0"/>
+        <origin xyz="0 ${distal_pad_box_y/2-0.002} ${-distal_pad_box_z/2+0.0005}" rpy="0 0 0"/>
         <mass value="${distal_pad_mass}"/>
-        <xacro:cuboid_inertia m="${distal_pad_mass}" x="0.005" y="0.15" z="0.039"/>
-      </inertial>
-      <collision>
-        <origin xyz="-0.00825 0.009 0.057" rpy="${pi/2} ${pi/2} 0"/>
+        <xacro:cuboid_inertia m="${distal_pad_mass}" x="${distal_pad_box_x}" y="${distal_pad_box_y}" z="${distal_pad_box_z}"/>
+      </inertial>
+      <collision>
+        <origin xyz="-0.009 0.0155 0.076" rpy="${pi/2} ${pi/2} 0"/>
         <geometry>
           <mesh filename="${mesh_path}/distal_pad_coll.STL"/>
@@ -149,4 +167,8 @@
     </link>
   </xacro:macro>
+  <!-- approx length, height and width of a cuboid surrounding the link -->
+  <xacro:property name="swivel_box_x" value="0.03"/>
+  <xacro:property name="swivel_box_y" value="0.03"/>
+  <xacro:property name="swivel_box_z" value="0.015"/>
   <xacro:macro name="swivel_link" params="finger_id">
     <link name="swivel_${finger_id}">
@@ -159,7 +181,7 @@
       </visual>
       <inertial>
-        <origin xyz="0 0 0" rpy="0 0 0"/>
+        <origin xyz="0 0 ${swivel_box_z/2}" rpy="0 0 0"/>
         <mass value="${swivel_link_mass}"/>
-        <xacro:cuboid_inertia m="${swivel_link_mass}" x="0.022" y="0.032" z="0.03"/>
+        <xacro:cuboid_inertia m="${swivel_link_mass}" x="${swivel_box_x}" y="${swivel_box_y}" z="${swivel_box_z}"/>
       </inertial>
       <collision>
@@ -171,4 +193,9 @@
     </link>
   </xacro:macro>
+  <!-- approx length, height and width of a cuboid surrounding the link -->
+  <xacro:property name="shell_box_x" value="0.13"/>
+  <xacro:property name="shell_box_y" value="0.09"/>
+  <xacro:property name="shell_box_z" value="0.07"/>
+  <xacro:property name="shell_x_offset" value="0.01"/>
   <xacro:macro name="shell_link">
     <link name="shell">
@@ -181,7 +208,7 @@
       </visual>
       <inertial>
-        <origin xyz="0 0 0" rpy="0 0 0"/>
+        <origin xyz="${shell_x_offset} 0 ${shell_box_z/2}" rpy="0 0 0"/>
         <mass value="${shell_mass}"/>
-        <xacro:cuboid_inertia m="${shell_mass}" x="0.066" y="0.091" z="0.136"/>
+        <xacro:cuboid_inertia m="${shell_mass}" x="${shell_box_x}" y="${shell_box_y}" z="${shell_box_z}"/>
       </inertial>
       <collision>
@@ -193,4 +220,6 @@
     </link>
   </xacro:macro>
+  <!-- y, z measurements we take from the shell -->
+  <xacro:property name="pad_box_y" value="0.022"/>
   <xacro:macro name="pad_link">
     <link name="pad">
@@ -203,7 +232,7 @@
       </visual>
       <inertial>
-        <origin xyz="0 0 0" rpy="0 0 0"/>
+        <origin xyz="0 ${pad_box_y/2} ${shell_x_offset}" rpy="0 0 0"/>
         <mass value="${pad_mass}"/>
-        <xacro:cuboid_inertia m="${pad_mass}" x="0.066" y="0.091" z="0.136"/>
+        <xacro:cuboid_inertia m="${pad_mass}" x="${shell_box_y}" y="${pad_box_y}" z="${shell_box_x}"/>
       </inertial>
       <collision>
@@ -215,5 +244,4 @@
     </link>
   </xacro:macro>
-  <link name="palm_link" />
   <!-- =================================== Tactile macros =================================== -->
   <!-- Sensor links are rendered only to give a link that the Gazebo sensor plugin can latch  -->
@@ -245,5 +273,4 @@
   <xacro:macro name="sensor_joint" params="location finger_id sensor_id">
     <joint name="${location}_${finger_id}_to_sensor_${sensor_id}" type="fixed">
-    <!-- TODO check why z_offset is different for distal and proximal  -->
       <xacro:if value="${location == 'proximal'}">
         <xacro:property name="x_offset" value="0.012"/>
@@ -252,7 +279,7 @@
       </xacro:if>
       <xacro:if value="${location == 'distal'}">
-        <xacro:property name="x_offset" value="0.008"/>
+        <xacro:property name="x_offset" value="-0.001"/>
         <xacro:property name="x_gap" value="0.008"/>
-        <xacro:property name="z_offset" value="0.01"/>
+        <xacro:property name="z_offset" value="0.0155"/>
       </xacro:if>
       <origin xyz="${x_offset + x_gap * sensor_id} 0 ${z_offset}" rpy="0 0 0"/>
@@ -261,14 +288,8 @@
     </joint>
   </xacro:macro>
-  <joint name="palm" type="fixed">
-    <origin xyz="0 0 0" rpy="3.14159265358979 0 1.5707963267949"/>
-    <parent link="pad" />
-    <child link="palm_link" />
-    <axis xyz="0 0 0"/>
-  </joint>
   <!-- ===================================== Joint Macros ===================================== -->
   <xacro:macro name="distal_to_pad" params="finger_id">
     <joint name="distal_${finger_id}_to_pad" type="fixed">
-      <origin xyz="-0.01 0 0.001" rpy="${pi/2} 0 -${pi/2}"/>
+      <origin xyz="0 0 0" rpy="${pi/2} 0 -${pi/2}"/>
       <parent link="distal_${finger_id}"/>
       <child link="distal_${finger_id}_pad"/>
@@ -283,15 +304,24 @@
   </xacro:macro>
   <xacro:macro name="flex_to_distal" params="finger_id">
-    <joint name="flex_to_distal_${finger_id}" type="fixed">
-      <origin xyz="0 0 0" rpy="0 0 0"/>
+    <joint name="flex_to_distal_${finger_id}" type="revolute">
+      <origin xyz="${flex_link_box_x} 0 0" rpy="0 0 0"/>
       <parent link="finger_${finger_id}_flex_link"/>
       <child link="distal_${finger_id}"/>
-    </joint>
-  </xacro:macro>
+      <axis xyz="0 -1 0"/>
+      <dynamics damping="0.0001" />
+      <!-- TODO might need to tune effort and velocity values -->
+      <limit effort="0.1" lower="0.0" upper="${pi/6}" velocity="1"/>
+    </joint>
+  </xacro:macro>
+  <xacro:property name="flex_z_offset" value="-0.002"/>
   <xacro:macro name="proximal_to_flex" params="finger_id">
-    <joint name="proximal_${finger_id}_to_flex" type="fixed">
-      <origin xyz="0.07 0 0.004" rpy="0 0 0"/>
+    <joint name="proximal_${finger_id}_to_flex" type="revolute">
+      <origin xyz="${0.0705-flex_link_box_x/2} 0 ${flex_z_offset}" rpy="0 0 0"/>
       <parent link="proximal_${finger_id}"/>
       <child link="finger_${finger_id}_flex_link"/>
+      <axis xyz="0 -1 0"/>
+      <dynamics damping="0.0001" />
+      <!-- TODO might need to tune effort and velocity values -->
+      <limit effort="0.1" lower="0.0" upper="${pi/6}" velocity="1"/>
     </joint>
   </xacro:macro>

Commit message: Tune effort values

File: simulation/description/urdf/reflex/reflex.urdf.xacro (robot description, xacro)
@@ -311,5 +311,5 @@
       <dynamics damping="0.0001" />
       <!-- TODO might need to tune effort and velocity values -->
-      <limit effort="0.1" lower="0.0" upper="${pi/6}" velocity="1"/>
+      <limit effort="1" lower="0.0" upper="${pi/6}" velocity="0.1"/>
     </joint>
   </xacro:macro>
@@ -323,5 +323,5 @@
       <dynamics damping="0.0001" />
       <!-- TODO might need to tune effort and velocity values -->
-      <limit effort="0.1" lower="0.0" upper="${pi/6}" velocity="1"/>
+      <limit effort="1" lower="0.0" upper="${pi/6}" velocity="0.1"/>
     </joint>
   </xacro:macro>
@@ -339,5 +339,5 @@
       <child link="swivel_${finger_id}"/>
       <dynamics damping="0.1" />
-      <limit effort="0.2" lower="0.0" upper="${pi/2}" velocity="0.01"/>
+      <limit effort="1" lower="0.0" upper="${pi/2}" velocity="0.1"/>
       <xacro:if value="${finger_id == 1}">
         <origin xyz="0.0503973683071414 -0.026 0.063" rpy="0 0 0"/>
@@ -355,5 +355,5 @@
       <axis xyz="0 -1 0"/>
       <dynamics damping="0.1" />
-      <limit effort="0.2" lower="0.0" upper="${pi}" velocity="0.01"/>
+      <limit effort="1" lower="0.0" upper="${pi}" velocity="0.1"/>
       <xacro:if value="${finger_id == 3}">
         <origin xyz="-0.03 0 0.0816" rpy="0 0.28 ${pi}"/>

Commit message: Increase flex link mass

File: simulation/description/urdf/reflex/reflex.urdf.xacro (robot description, xacro)
@@ -27,5 +27,5 @@
   <!-- ======================================= Masses ======================================== -->
   <!-- These are rough approximations, the total hand mass was measured to be about 0.9kg     -->
-  <!-- final mass: 0.6+0.03+2*0.02+3*(0.025+0.015+0.01+0.02+0.01) = 0.91 -->
+  <!-- final mass: 0.6+0.03+2*0.02+3*(0.025+0.015+0.02+0.02+0.01) = 0.94 -->
   <xacro:property name="shell_mass" value="0.6"/>
   <xacro:property name="pad_mass" value="0.03"/>
@@ -35,5 +35,5 @@
   <xacro:property name="proximal_link_mass" value="0.025"/>
   <xacro:property name="proximal_pad_mass" value="0.015"/>
-  <xacro:property name="flex_link_mass" value="0.01"/>
+  <xacro:property name="flex_link_mass" value="0.02"/>
   <xacro:property name="distal_link_mass" value="0.02"/>
   <xacro:property name="distal_pad_mass" value="0.01"/>

Commit message: Update effort/damping/velocities for DART engine

File: simulation/description/urdf/reflex/reflex.urdf.xacro (robot description, xacro)
@@ -250,4 +250,8 @@
   <!-- enough not to interfere with the hand dynamics, but not so small that they physics     -->
   <!-- engine chokes on it (e.g. 1e-8 is too small and the links disappear).                  -->
+  <xacro:property name="sensor_box_x" value="0.006"/>
+  <xacro:property name="sensor_box_y" value="0.006"/>
+  <xacro:property name="sensor_box_z" value="0.0003"/>
+  <xacro:property name="sensor_mass" value="1e-5"/>
   <xacro:macro name="sensor_link" params="location finger_id sensor_id">
     <link name="${location}_${finger_id}_sensor_${sensor_id}">
@@ -255,16 +259,16 @@
         <origin xyz="0 0 0" rpy="0 0 0"/>
         <geometry>
-          <box size="0.006 0.006 0.0003"/>
-        </geometry>
-      </visual>
-      <inertial>
-        <origin xyz="0 0 0" rpy="0 0 0"/>
-        <mass value="1e-5"/>
-        <xacro:cuboid_inertia m="1e-5" x="0.006" y="0.006" z="0.0003"/>
-      </inertial>
-      <collision>
-        <origin xyz="0 0 0" rpy="0 0 0"/>
-        <geometry>
-          <box size="0.006 0.006 0.0003"/>
+          <box size="${sensor_box_x} ${sensor_box_y} ${sensor_box_z}"/>
+        </geometry>
+      </visual>
+      <inertial>
+        <origin xyz="0 0 0" rpy="0 0 0"/>
+        <mass value="${sensor_mass}"/>
+        <xacro:cuboid_inertia m="${sensor_mass}" x="${sensor_box_x}" y="${sensor_box_y}" z="${sensor_box_z}"/>
+      </inertial>
+      <collision>
+        <origin xyz="0 0 0" rpy="0 0 0"/>
+        <geometry>
+          <box size="${sensor_box_x} ${sensor_box_y} ${sensor_box_z}"/>
         </geometry>
       </collision>
@@ -309,7 +313,7 @@
       <child link="distal_${finger_id}"/>
       <axis xyz="0 -1 0"/>
-      <dynamics damping="0.0001" />
-      <!-- TODO might need to tune effort and velocity values -->
-      <limit effort="1" lower="0.0" upper="${pi/6}" velocity="0.1"/>
+      <!-- note: I estimate the remaining damping/effort/velocity is half of the proximal links -->
+      <dynamics damping="0.05" friction="0"/>
+      <limit effort="1" lower="0.0" upper="${pi/6}" velocity="0.5"/>
     </joint>
   </xacro:macro>
@@ -321,7 +325,7 @@
       <child link="finger_${finger_id}_flex_link"/>
       <axis xyz="0 -1 0"/>
-      <dynamics damping="0.0001" />
-      <!-- TODO might need to tune effort and velocity values -->
-      <limit effort="1" lower="0.0" upper="${pi/6}" velocity="0.1"/>
+      <!-- note: I estimate the remaining damping/effort/velocity is half of the proximal links -->
+      <dynamics damping="0.05" friction="0"/>
+      <limit effort="1" lower="0.0" upper="${pi/6}" velocity="0.5"/>
     </joint>
   </xacro:macro>
@@ -335,9 +339,11 @@
   </xacro:macro>
   <xacro:macro name="preshape" params="finger_id">
-    <joint name="preshape_${finger_id}" type="${joint_type}">
+    <joint name="preshape_${finger_id}" type="revolute">
       <parent link="shell"/>
       <child link="swivel_${finger_id}"/>
-      <dynamics damping="0.1" />
-      <limit effort="1" lower="0.0" upper="${pi/2}" velocity="0.1"/>
+      <!-- damping factor of 0.1 makes the joint move smoother -->
+      <dynamics damping="0.1" friction="0"/>
+      <!-- note: the dynamixel motors can apply roughly 2Nm (see datasheet) -->
+      <limit effort="2" lower="0.0" upper="${pi/2}" velocity="1"/>
       <xacro:if value="${finger_id == 1}">
         <origin xyz="0.0503973683071414 -0.026 0.063" rpy="0 0 0"/>
@@ -351,9 +357,11 @@
   </xacro:macro>
   <xacro:macro name="proximal" params="finger_id">
-    <joint name="proximal_joint_${finger_id}" type="${joint_type}">
+    <joint name="proximal_joint_${finger_id}" type="revolute">
       <child link="proximal_${finger_id}"/>
       <axis xyz="0 -1 0"/>
-      <dynamics damping="0.1" />
-      <limit effort="1" lower="0.0" upper="${pi}" velocity="0.1"/>
+      <!-- damping factor of 0.1 makes the joint move smoother -->
+      <dynamics damping="0.1" friction="0"/>
+      <!-- note: the dynamixel motors can apply roughly 2Nm (see datasheet) -->
+      <limit effort="2" lower="0.0" upper="${pi}" velocity="1"/>
       <xacro:if value="${finger_id == 3}">
         <origin xyz="-0.03 0 0.0816" rpy="0 0.28 ${pi}"/>
