Commit message: Remove visual & collision elements from wrist urdf

File: simulation/wrist_controller/urdf/wrist.urdf.xacro (robot description, xacro)
@@ -12,9 +12,6 @@
     <xacro:property name="rotation_damping" value="0"/>
     <xacro:property name="rotation_friction" value="0"/>
-    <link name="base_footprint" />
-    <!-- this all comes from grasp repo -->
-    <!-- Virtual link world -->
+    <!-- links and joints for translation -->
     <link name="world"/>
-    <!-- Translation -->
     <joint name="virtual_px_joint" type="prismatic">
         <origin rpy="0 0 0" xyz="0 0 0"/>
@@ -26,10 +23,4 @@
     </joint>
     <link name="virtual_px_link">
-        <visual>
-            <origin rpy="0 0 0" xyz="0 0 0"/>
-            <geometry>
-                <cylinder length="0.01" radius="0.005"/>
-            </geometry>
-        </visual>
         <inertial>
             <origin rpy="0 0 0" xyz="0 0 0"/>
@@ -37,10 +28,4 @@
             <inertia ixx="0.01" ixy="0" ixz="0" iyy="0.01" iyz="0" izz="0.01"/>
         </inertial>
-        <collision>
-            <origin rpy="0 0 0" xyz="0.0 0.0 -20.0"/>
-            <geometry>
-                <cylinder length="0.001" radius="0.005"/>
-            </geometry>
-        </collision>
     </link>
     <joint name="virtual_py_joint" type="prismatic">
@@ -53,10 +38,4 @@
     </joint>
     <link name="virtual_py_link">
-        <visual>
-            <origin rpy="0 0 0" xyz="0 0 0"/>
-            <geometry>
-                <cylinder length="0.01" radius="0.005"/>
-            </geometry>
-        </visual>
         <inertial>
             <origin rpy="0 0 0" xyz="0 0 0"/>
@@ -64,10 +43,4 @@
             <inertia ixx="0.01" ixy="0" ixz="0" iyy="0.01" iyz="0" izz="0.01"/>
         </inertial>
-        <collision>
-            <origin rpy="0 0 0" xyz="0.0 0.0 -20.0"/>
-            <geometry>
-                <cylinder length="0.001" radius="0.005"/>
-            </geometry>
-        </collision>
     </link>
     <joint name="virtual_pz_joint" type="prismatic">
@@ -80,10 +53,4 @@
     </joint>
     <link name="virtual_pz_link">
-        <visual>
-            <origin rpy="0 0 0" xyz="0 0 0"/>
-            <geometry>
-                <cylinder length="0.01" radius="0.005"/>
-            </geometry>
-        </visual>
         <inertial>
             <origin rpy="0 0 0" xyz="0 0 0"/>
@@ -91,12 +58,6 @@
             <inertia ixx="0.01" ixy="0" ixz="0" iyy="0.01" iyz="0" izz="0.01"/>
         </inertial>
-        <collision>
-            <origin rpy="0 0 0" xyz="0.0 0.0 -20.0"/>
-            <geometry>
-                <cylinder length="0.001" radius="0.005"/>
-            </geometry>
-        </collision>
     </link>
-    <!-- Rotation -->
+    <!-- links and joints for rotation -->
     <joint name="virtual_ry_joint" type="continuous">
         <origin rpy="0 0 0" xyz="0 0 0"/>
@@ -108,10 +69,4 @@
     </joint>
     <link name="virtual_ry_link">
-        <visual>
-            <origin rpy="0 0 0" xyz="0 0 0"/>
-            <geometry>
-                <cylinder length="0.01" radius="0.005"/>
-            </geometry>
-        </visual>
         <inertial>
             <origin rpy="0 0 0" xyz="0 0 0"/>
@@ -119,10 +74,4 @@
             <inertia ixx="0.01" ixy="0" ixz="0" iyy="0.01" iyz="0" izz="0.01"/>
         </inertial>
-        <collision>
-            <origin rpy="0 0 0" xyz="0.0 0.0 -20.0"/>
-            <geometry>
-                <cylinder length="0.001" radius="0.005"/>
-            </geometry>
-        </collision>
     </link>
     <joint name="virtual_rp_joint" type="continuous">
@@ -135,10 +84,4 @@
     </joint>
     <link name="virtual_rp_link">
-        <visual>
-            <origin rpy="0 0 0" xyz="0 0 0"/>
-            <geometry>
-                <cylinder length="0.01" radius="0.005"/>
-            </geometry>
-        </visual>
         <inertial>
             <origin rpy="0 0 0" xyz="0 0 0"/>
@@ -146,23 +89,13 @@
             <inertia ixx="0.01" ixy="0" ixz="0" iyy="0.01" iyz="0" izz="0.01"/>
         </inertial>
-        <collision>
-            <origin rpy="0 0 0" xyz="0.0 0.0 -20.0"/>
-            <geometry>
-                <cylinder length="0.001" radius="0.005"/>
-            </geometry>
-        </collision>
     </link>
+    <!-- if you want to use this package with other robot hands, simply replace the "shell" link with the base link of your robot hand -->
     <joint name="virtual_rr_joint" type="continuous">
         <origin rpy="0 0 0" xyz="0 0 0"/>
         <axis xyz="1 0 0"/>
         <parent link="virtual_rp_link"/>
-        <child link="base_footprint"/>
+        <child link="shell"/>
         <limit effort="${rotation_effort}" velocity="${rotation_velocity}"/>
         <dynamics damping="${rotation_damping}" friction="${rotation_friction}"/>
-    </joint>
-    <!-- if you want to use this package with other robot hands, simply replace the "shell" link with the base link of your robot hand -->
-    <joint name="base_to_shell_joint" type="fixed">
-        <parent link="base_footprint" />
-        <child link = "shell" />
     </joint>
     <!-- transmissions -->

Commit message: Tune damping coefficients

File: simulation/wrist_controller/urdf/wrist.urdf.xacro (robot description, xacro)
@@ -6,9 +6,10 @@
     <xacro:property name="translation_up_lim" value="5"/>
     <xacro:property name="translation_low_lim" value="-5"/>
-    <xacro:property name="translation_damping" value="30"/>
+    <xacro:property name="translation_damping" value="60"/>
+    <xacro:property name="translation_friction" value="0"/>
     <!-- rotation properties -->
     <xacro:property name="rotation_effort" value="1000"/>
     <xacro:property name="rotation_velocity" value="25"/>
-    <xacro:property name="rotation_damping" value="0"/>
+    <xacro:property name="rotation_damping" value="60"/>
     <xacro:property name="rotation_friction" value="0"/>
     <!-- links and joints for translation -->
@@ -20,5 +21,5 @@
         <child link="virtual_px_link"/>
         <limit effort="${translation_effort}" lower="${translation_low_lim}" upper="${translation_up_lim}" velocity="${translation_velocity}"/>
-        <dynamics damping="${translation_damping}"/>
+        <dynamics damping="${translation_damping}" friction="${translation_friction}"/>
     </joint>
     <link name="virtual_px_link">
@@ -35,5 +36,5 @@
         <child link="virtual_py_link"/>
         <limit effort="${translation_effort}" lower="${translation_low_lim}" upper="${translation_up_lim}" velocity="${translation_velocity}"/>
-        <dynamics damping="${translation_damping}"/>
+        <dynamics damping="${translation_damping}" friction="${translation_friction}"/>
     </joint>
     <link name="virtual_py_link">
@@ -50,5 +51,5 @@
         <child link="virtual_pz_link"/>
         <limit effort="${translation_effort}" lower="${translation_low_lim}" upper="${translation_up_lim}" velocity="${translation_velocity}"/>
-        <dynamics damping="${translation_damping}"/>
+        <dynamics damping="${translation_damping}" friction="${translation_friction}"/>
     </joint>
     <link name="virtual_pz_link">

Commit message: Outsource hard coded values

File: simulation/wrist_controller/urdf/wrist.urdf.xacro (robot description, xacro)
@@ -66,6 +66,6 @@
         <parent link="virtual_pz_link"/>
         <child link="virtual_ry_link"/>
-        <limit effort="50.00" velocity="25.0"/>
-        <dynamics damping="100.0" friction="5.0"/>
+        <limit effort="${rotation_effort}" velocity="${rotation_velocity}"/>
+        <dynamics damping="${rotation_damping}" friction="${rotation_friction}"/>
     </joint>
     <link name="virtual_ry_link">

Commit message: Limit velocity

File: simulation/wrist_controller/urdf/wrist.urdf.xacro (robot description, xacro)
@@ -3,5 +3,5 @@
     <!-- translation properties -->
     <xacro:property name="translation_effort" value="1000"/>
-    <xacro:property name="translation_velocity" value="25"/>
+    <xacro:property name="translation_velocity" value="0.5"/>
     <xacro:property name="translation_up_lim" value="5"/>
     <xacro:property name="translation_low_lim" value="-5"/>
@@ -10,5 +10,5 @@
     <!-- rotation properties -->
     <xacro:property name="rotation_effort" value="1000"/>
-    <xacro:property name="rotation_velocity" value="25"/>
+    <xacro:property name="rotation_velocity" value="0.1"/>
     <xacro:property name="rotation_damping" value="60"/>
     <xacro:property name="rotation_friction" value="0"/>
