Commit message: Add box and cylinder support

File: simulation/description/urdf/environment/box.urdf.xacro (robot description, xacro)
@@ -1,28 +1,32 @@
 <?xml version="1.0" encoding="UTF-8"?>
 <robot xmlns:xacro="http://ros.org/wiki/xacro" name="box">
-  <link name="box_link">
-    <inertial>
-      <origin xyz="0 0 0" rpy="0 0 0"/>
-      <mass value="0.01"/>
-      <inertia ixx="1e-3"  ixy="0"  ixz="0" iyy="1e-3" iyz="0" izz="1e-3" />
-    </inertial>
-    <visual>
-      <origin xyz="0 0 0" rpy="0 0 0" />
-      <geometry>
-	<box size="0.05 0.05 0.05" />
-      </geometry>
-      <material name="green">
-	<color rgba="0 0.6 0.6 1"/>
-      </material>
-    </visual>
-    <collision>
-      <origin xyz="0 0 0" rpy="0 0 0" />
-      <geometry>
-	<box size="0.05 0.05 0.05" />
-      </geometry>
-    </collision>
-  </link>
-  <gazebo reference="box_link">
-    <material>Gazebo/Blue</material>
-  </gazebo>
+    <!-- arguments -->
+    <xacro:arg name="box_mass" default="0.2"/>
+    <xacro:arg name="box_inertia" default="0.0006"/>
+    <xacro:arg name="box_x" default="0.08"/>
+    <xacro:arg name="box_y" default="0.08"/>
+    <xacro:arg name="box_z" default="0.08"/>
+    <xacro:property name="link_name" value="box_link"/>
+    <link name="${link_name}">
+        <visual>
+            <origin xyz="0 0 0" rpy="0 0 0" />
+            <geometry>
+                <box size="$(arg box_x) $(arg box_y) $(arg box_z)" />
+            </geometry>
+        </visual>
+        <collision>
+            <origin xyz="0 0 0" rpy="0 0 0" />
+            <geometry>
+                <box size="$(arg box_x) $(arg box_y) $(arg box_z)" />
+            </geometry>
+        </collision>
+        <inertial>
+            <origin xyz="0 0 0" rpy="0 0 0"/>
+            <mass value="$(arg box_mass)"/>
+            <inertia ixx="$(arg box_inertia)" ixy="0" ixz="0" iyy="$(arg box_inertia)" iyz="0" izz="$(arg box_inertia)" />
+        </inertial>
+    </link>
+    <gazebo reference="${link_name}">
+        <material>Gazebo/Green</material>
+    </gazebo>
 </robot>

File: simulation/description/urdf/environment/sphere.urdf.xacro (robot description, xacro)
@@ -2,14 +2,13 @@
 <robot xmlns:xacro="http://ros.org/wiki/xacro" name="sphere">
     <!-- arguments -->
-    <xacro:arg name="object_height" default="0.17"/>
     <xacro:arg name="sphere_mass" default="0.2"/>
     <xacro:arg name="sphere_inertia" default="0.0006"/>
+    <xacro:arg name="sphere_radius" default="0.08"/>
     <xacro:property name="link_name" value="sphere_link"/>
-    <xacro:property name="sphere_radius" value="${$(arg object_height)/2}"/>
     <link name="${link_name}">
         <visual>
             <origin xyz="0 0 0" rpy="0 0 0" />
             <geometry>
-                <sphere radius="${sphere_radius}" />
+                <sphere radius="$(arg sphere_radius)" />
             </geometry>
         </visual>
@@ -17,5 +16,5 @@
             <origin xyz="0 0 0" rpy="0 0 0" />
             <geometry>
-                <sphere radius="${sphere_radius}" />
+                <sphere radius="$(arg sphere_radius)" />
             </geometry>
         </collision>

Commit message: Add sensor plugin to object to obtain contact info

File: simulation/description/urdf/environment/box.urdf.xacro (robot description, xacro)
@@ -27,6 +27,4 @@
         </inertial>
     </link>
-    <gazebo reference="${link_name}">
-        <material>Gazebo/Green</material>
-    </gazebo>
+    <xacro:include filename="$(find description)/urdf/environment/object.gazebo.xacro"/>
 </robot>

File: simulation/description/urdf/environment/cylinder.urdf.xacro (robot description, xacro)
@@ -26,6 +26,4 @@
         </inertial>
     </link>
-    <gazebo reference="${link_name}">
-        <material>Gazebo/Green</material>
-    </gazebo>
+    <xacro:include filename="$(find description)/urdf/environment/object.gazebo.xacro"/>
 </robot>

File: simulation/description/urdf/environment/sphere.urdf.xacro (robot description, xacro)
@@ -25,6 +25,4 @@
         </inertial>
     </link>
-    <gazebo reference="${link_name}">
-        <material>Gazebo/Green</material>
-    </gazebo>
+    <xacro:include filename="$(find description)/urdf/environment/object.gazebo.xacro"/>
 </robot>
