Commit message: Add preserve fixed joint tag

File: reflex_stack/simulation/description/urdf/reflex/reflex.gazebo.xacro (robot description, xacro)
@@ -63,5 +63,5 @@
   <!-- adds sensor plugin to proximal and distal links -->
   <xacro:macro name="link_sensor" params="location finger_id">
-    <xacro:property name="link_name" value="${location}_${finger_id}"/>
+    <xacro:property name="link_name" value="${location}_${finger_id}_pad"/>
     <xacro:property name="sensor_name" value="gazebo/${link_name}_sensor"/>
     <gazebo reference="${link_name}">
@@ -81,4 +81,12 @@
   <xacro:macro name="preserve_fixed" params="location finger_id sensor_id">
     <gazebo reference="${location}_${finger_id}_to_sensor_${sensor_id}">
+      <preserveFixedJoint>true</preserveFixedJoint>
+    </gazebo>
+  </xacro:macro>
+  <!-- this makes sure that link stays seperate from parent link. by default
+       Gazebo merges links with fixed joints together to one link, but here
+       we need it to be separate to latch on the libgazebo_ros_bumper plugin -->
+  <xacro:macro name="preserve_fixed_pad" params="location finger_id">
+    <gazebo reference="${location}_${finger_id}_to_pad">
       <preserveFixedJoint>true</preserveFixedJoint>
     </gazebo>
@@ -111,4 +119,6 @@
     <xacro:preserve_fixed location="distal" finger_id="${id}" sensor_id="3"/>
     <xacro:preserve_fixed location="distal" finger_id="${id}" sensor_id="4"/>
+    <xacro:preserve_fixed_pad location="proximal" finger_id="${id}"/>
+    <xacro:preserve_fixed_pad location="distal" finger_id="${id}"/>
   </xacro:macro>
   <xacro:gazebo_finger id="1"/>

Commit message: Add Gazebo sensor to palm pad

File: reflex_stack/simulation/description/urdf/reflex/reflex.gazebo.xacro (robot description, xacro)
@@ -61,7 +61,6 @@
     </gazebo>
   </xacro:macro>
-  <!-- adds sensor plugin to proximal and distal links -->
-  <xacro:macro name="link_sensor" params="location finger_id">
-    <xacro:property name="link_name" value="${location}_${finger_id}_pad"/>
+  <!-- adds sensor plugin to links -->
+  <xacro:macro name="link_sensor" params="link_name">
     <xacro:property name="sensor_name" value="gazebo/${link_name}_sensor"/>
     <gazebo reference="${link_name}">
@@ -108,6 +107,6 @@
     <xacro:tactile_sensor location="distal" finger_id="${id}" sensor_id="3"/>
     <xacro:tactile_sensor location="distal" finger_id="${id}" sensor_id="4"/>
-    <xacro:link_sensor location="proximal" finger_id="${id}"/>
-    <xacro:link_sensor location="distal" finger_id="${id}"/>
+    <xacro:link_sensor link_name="proximal_${id}"/>
+    <xacro:link_sensor link_name="distal_${id}"/>
     <xacro:preserve_fixed location="proximal" finger_id="${id}" sensor_id="1"/>
     <xacro:preserve_fixed location="proximal" finger_id="${id}" sensor_id="2"/>
@@ -125,3 +124,8 @@
   <xacro:gazebo_finger id="2"/>
   <xacro:gazebo_finger id="3"/>
+  <!-- latch sensor onto palm pad -->
+  <xacro:link_sensor link_name="pad"/>
+  <gazebo reference="shell_to_pad">
+    <preserveFixedJoint>true</preserveFixedJoint>
+  </gazebo>
 </robot>
