Commit message: Make sensors even bigger

File: reflex_stack/simulation/description/urdf/reflex/reflex.urdf.xacro (robot description, xacro)
@@ -250,7 +250,8 @@
   <!-- enough not to interfere with the hand dynamics, but not so small that they physics     -->
   <!-- engine chokes on it (e.g. 1e-8 is too small and the links disappear).                  -->
-  <xacro:property name="sensor_box_x" value="0.008"/>
-  <xacro:property name="sensor_box_y" value="0.009"/>
-  <xacro:property name="sensor_box_z" value="0.0003"/>
+  <xacro:property name="sensor_box_x_proximal" value="0.0099"/>
+  <xacro:property name="sensor_box_x_distal" value="0.0092"/>
+  <xacro:property name="sensor_box_y" value="0.015"/>
+  <xacro:property name="sensor_box_z" value="0.006"/>
   <xacro:property name="sensor_mass" value="1e-5"/>
   <xacro:macro name="sensor_link" params="location finger_id sensor_id">
@@ -259,5 +260,10 @@
         <origin xyz="0 0 0" rpy="0 0 0"/>
         <geometry>
-          <box size="${sensor_box_x} ${sensor_box_y} ${sensor_box_z}"/>
+          <xacro:if value="${location == 'proximal'}">
+            <box size="${sensor_box_x_proximal} ${sensor_box_y} ${sensor_box_z}"/>
+          </xacro:if>
+          <xacro:if value="${location == 'distal'}">
+            <box size="${sensor_box_x_distal} ${sensor_box_y} ${sensor_box_z}"/>
+          </xacro:if>
         </geometry>
       </visual>
@@ -265,10 +271,20 @@
         <origin xyz="0 0 0" rpy="0 0 0"/>
         <mass value="${sensor_mass}"/>
-        <xacro:cuboid_inertia m="${sensor_mass}" x="${sensor_box_x}" y="${sensor_box_y}" z="${sensor_box_z}"/>
-      </inertial>
-      <collision>
-        <origin xyz="0 0 0" rpy="0 0 0"/>
-        <geometry>
-          <box size="${sensor_box_x} ${sensor_box_y} ${sensor_box_z}"/>
+          <xacro:if value="${location == 'proximal'}">
+            <xacro:cuboid_inertia m="${sensor_mass}" x="${sensor_box_x_proximal}" y="${sensor_box_y}" z="${sensor_box_z}"/>
+          </xacro:if>
+          <xacro:if value="${location == 'distal'}">
+            <xacro:cuboid_inertia m="${sensor_mass}" x="${sensor_box_x_distal}" y="${sensor_box_y}" z="${sensor_box_z}"/>
+          </xacro:if>
+      </inertial>
+      <collision>
+        <origin xyz="0 0 0" rpy="0 0 0"/>
+        <geometry>
+          <xacro:if value="${location == 'proximal'}">
+            <box size="${sensor_box_x_proximal} ${sensor_box_y} ${sensor_box_z}"/>
+          </xacro:if>
+          <xacro:if value="${location == 'distal'}">
+            <box size="${sensor_box_x_distal} ${sensor_box_y} ${sensor_box_z}"/>
+          </xacro:if>
         </geometry>
       </collision>
@@ -278,12 +294,12 @@
     <joint name="${location}_${finger_id}_to_sensor_${sensor_id}" type="fixed">
       <xacro:if value="${location == 'proximal'}">
-        <xacro:property name="x_offset" value="0.012"/>
-        <xacro:property name="x_gap" value="0.008"/>
-        <xacro:property name="z_offset" value="0.014"/>
+        <xacro:property name="x_offset" value="0.008"/>
+        <xacro:property name="x_gap" value="0.0097"/>
+        <xacro:property name="z_offset" value="${0.014-sensor_box_z/2}"/>
       </xacro:if>
       <xacro:if value="${location == 'distal'}">
-        <xacro:property name="x_offset" value="-0.001"/>
-        <xacro:property name="x_gap" value="0.008"/>
-        <xacro:property name="z_offset" value="0.0155"/>
+        <xacro:property name="x_offset" value="-0.004"/>
+        <xacro:property name="x_gap" value="0.0091"/>
+        <xacro:property name="z_offset" value="${0.0155-sensor_box_z/2}"/>
       </xacro:if>
       <origin xyz="${x_offset + x_gap * sensor_id} 0 ${z_offset}" rpy="0 0 0"/>

Commit message: Simplify collision meshes

File: reflex_stack/simulation/description/urdf/reflex/reflex.urdf.xacro (robot description, xacro)
@@ -2,5 +2,7 @@
 <robot xmlns:xacro="http://www.ros.org/wiki/xacro" name="reflex">
   <xacro:arg name="actuate_reflex" default="true"/>
-  <xacro:arg name="use_reflex_contact_sensors" default="true"/>
+  <xacro:arg name="use_reflex_contact_sensors" default="false"/>
+  <!-- removes all unnecessary collision meshes for grasping and turns necessary ones into boxes -->
+  <xacro:arg name="simplify_collisions" default="false"/>
   <!-- Switch joint type for actuated joints depending on if they are being used for control -->
   <xacro:if value="$(arg actuate_reflex)">
@@ -56,10 +58,12 @@
         <xacro:cuboid_inertia m="${flex_link_mass}" x="${flex_link_box_x}" y="${flex_link_box_y}" z="${flex_link_box_z}"/>
       </inertial>
-      <collision>
-        <origin xyz="${flex_link_box_x/2} 0 ${flex_link_box_z/2}" rpy="0 0 0"/>
-        <geometry>
-          <box size="${flex_link_box_x} ${flex_link_box_y} ${flex_link_box_z}"/>
-        </geometry>
-      </collision>
+      <xacro:unless value="$(arg simplify_collisions)">
+        <collision>
+          <origin xyz="${flex_link_box_x/2} 0 ${flex_link_box_z/2}" rpy="0 0 0"/>
+          <geometry>
+            <box size="${flex_link_box_x} ${flex_link_box_y} ${flex_link_box_z}"/>
+          </geometry>
+        </collision>
+      </xacro:unless>
     </link>
   </xacro:macro>
@@ -82,10 +86,12 @@
         <xacro:cuboid_inertia m="${proximal_link_mass}" x="${proximal_link_box_x}" y="${proximal_link_box_y}" z="${proximal_link_box_z}"/>
       </inertial>
-      <collision>
-        <origin xyz="-0.011 0.007 0.011" rpy="${pi} 0 0"/>
-        <geometry>
-          <mesh filename="${mesh_path}/proximal_coll.STL"/>
-        </geometry>
-      </collision>
+      <xacro:unless value="$(arg simplify_collisions)">
+        <collision>
+          <origin xyz="-0.011 0.007 0.011" rpy="${pi} 0 0"/>
+          <geometry>
+            <mesh filename="${mesh_path}/proximal_coll.STL"/>
+          </geometry>
+        </collision>
+      </xacro:unless>
     </link>
   </xacro:macro>
@@ -108,15 +114,17 @@
         <xacro:cuboid_inertia m="${distal_link_mass}" x="${distal_link_box_x}" y="${distal_link_box_y}" z="${distal_link_box_z}"/>
       </inertial>
-      <collision>
-        <origin xyz="${-0.077-flex_link_box_x/2} 0.007 ${0.007+flex_link_box_z/2}" rpy="${pi} 0 0"/>
-        <geometry>
-          <mesh filename="${mesh_path}/distal_coll.STL"/>
-        </geometry>
-      </collision>
+      <xacro:unless value="$(arg simplify_collisions)">
+        <collision>
+          <origin xyz="${-0.077-flex_link_box_x/2} 0.007 ${0.007+flex_link_box_z/2}" rpy="${pi} 0 0"/>
+          <geometry>
+            <mesh filename="${mesh_path}/distal_coll.STL"/>
+          </geometry>
+        </collision>
+      </xacro:unless>
     </link>
   </xacro:macro>
   <xacro:property name="proximal_pad_box_x" value="0.016"/>
   <xacro:property name="proximal_pad_box_y" value="0.020"/>
-  <xacro:property name="proximal_pad_box_z" value="0.05"/>
+  <xacro:property name="proximal_pad_box_z" value="0.052"/>
   <xacro:macro name="proximal_pad" params="finger_id">
     <link name="proximal_${finger_id}_pad">
@@ -134,8 +142,16 @@
       </inertial>
       <collision>
-        <origin xyz="-0.008 0.014 -0.002" rpy="${pi/2} ${pi/2} 0"/>
-        <geometry>
-          <mesh filename="${mesh_path}/proximal_pad_coll.STL"/>
-        </geometry>
+        <xacro:unless value="$(arg simplify_collisions)">
+          <origin xyz="-0.008 0.014 -0.002" rpy="${pi/2} ${pi/2} 0"/>
+          <geometry>
+            <mesh filename="${mesh_path}/proximal_pad_coll.STL"/>
+          </geometry>
+        </xacro:unless>
+        <xacro:if value="$(arg simplify_collisions)">
+          <origin xyz="0 0.004 -0.035" rpy="0 0 0"/>
+          <geometry>
+            <box size="${proximal_pad_box_x} ${proximal_pad_box_y} ${proximal_pad_box_z}"/>
+          </geometry>
+        </xacro:if>
       </collision>
     </link>
@@ -143,5 +159,5 @@
   <xacro:property name="distal_pad_box_x" value="${proximal_pad_box_x}"/>
   <xacro:property name="distal_pad_box_y" value="0.018"/>
-  <xacro:property name="distal_pad_box_z" value="0.037"/>
+  <xacro:property name="distal_pad_box_z" value="0.0385"/>
   <xacro:macro name="distal_pad" params="finger_id">
     <link name="distal_${finger_id}_pad">
@@ -160,8 +176,16 @@
       </inertial>
       <collision>
-        <origin xyz="-0.009 0.0155 0.076" rpy="${pi/2} ${pi/2} 0"/>
-        <geometry>
-          <mesh filename="${mesh_path}/distal_pad_coll.STL"/>
-        </geometry>
+        <xacro:unless value="$(arg simplify_collisions)">
+          <origin xyz="-0.008 0.0155 0.076" rpy="${pi/2} ${pi/2} 0"/>
+          <geometry>
+            <mesh filename="${mesh_path}/distal_pad_coll.STL"/>
+          </geometry>
+        </xacro:unless>
+        <xacro:if value="$(arg simplify_collisions)">
+          <origin xyz="0 ${distal_pad_box_y/2-0.002} ${-distal_pad_box_z/2+0.0005}" rpy="0 0 0"/>
+          <geometry>
+            <box size="${distal_pad_box_x} ${distal_pad_box_y} ${distal_pad_box_z}"/>
+          </geometry>
+        </xacro:if>
       </collision>
     </link>
@@ -185,10 +209,12 @@
         <xacro:cuboid_inertia m="${swivel_link_mass}" x="${swivel_box_x}" y="${swivel_box_y}" z="${swivel_box_z}"/>
       </inertial>
-      <collision>
-        <origin xyz="0 0 0" rpy="0 0 0"/>
-        <geometry>
-          <mesh filename="${mesh_path}/swivel_${finger_id}_coll.STL"/>
-        </geometry>
-      </collision>
+      <xacro:unless value="$(arg simplify_collisions)">
+        <collision>
+          <origin xyz="0 0 0" rpy="0 0 0"/>
+          <geometry>
+            <mesh filename="${mesh_path}/swivel_${finger_id}_coll.STL"/>
+          </geometry>
+        </collision>
+      </xacro:unless>
     </link>
   </xacro:macro>
@@ -212,14 +238,17 @@
         <xacro:cuboid_inertia m="${shell_mass}" x="${shell_box_x}" y="${shell_box_y}" z="${shell_box_z}"/>
       </inertial>
-      <collision>
-        <origin xyz="0 0 0" rpy="0 0 0"/>
-        <geometry>
-          <mesh filename="${mesh_path}/base_link_coll.STL"/>
-        </geometry>
-      </collision>
+      <xacro:unless value="$(arg simplify_collisions)">
+        <collision>
+          <origin xyz="0 0 0" rpy="0 0 0"/>
+          <geometry>
+            <mesh filename="${mesh_path}/base_link_coll.STL"/>
+          </geometry>
+        </collision>
+      </xacro:unless>
     </link>
   </xacro:macro>
   <!-- y, z measurements we take from the shell -->
   <xacro:property name="pad_box_y" value="0.022"/>
+  <xacro:property name="pad_x_offset" value="0.005"/>
   <xacro:macro name="pad_link">
     <link name="pad">
@@ -232,13 +261,21 @@
       </visual>
       <inertial>
-        <origin xyz="0 ${pad_box_y/2} ${shell_x_offset}" rpy="0 0 0"/>
+        <origin xyz="0 ${pad_box_y/2} ${pad_x_offset}" rpy="0 0 0"/>
         <mass value="${pad_mass}"/>
         <xacro:cuboid_inertia m="${pad_mass}" x="${shell_box_y}" y="${pad_box_y}" z="${shell_box_x}"/>
       </inertial>
       <collision>
-        <origin xyz="0 0 0" rpy="0 0 0"/>
-        <geometry>
-          <mesh filename="${mesh_path}/pad_coll.STL"/>
-        </geometry>
+        <xacro:unless value="$(arg simplify_collisions)">
+          <origin xyz="0 0 0" rpy="0 0 0"/>
+          <geometry>
+            <mesh filename="${mesh_path}/pad_coll.STL"/>
+          </geometry>
+        </xacro:unless>
+        <xacro:if value="$(arg simplify_collisions)">
+          <origin xyz="0 ${pad_box_y/2} ${pad_x_offset}" rpy="0 0 0"/>
+          <geometry>
+            <box size="${shell_box_y} ${pad_box_y} ${shell_box_x}"/>
+          </geometry>
+        </xacro:if>
       </collision>
     </link>
@@ -271,10 +308,10 @@
         <origin xyz="0 0 0" rpy="0 0 0"/>
         <mass value="${sensor_mass}"/>
-          <xacro:if value="${location == 'proximal'}">
-            <xacro:cuboid_inertia m="${sensor_mass}" x="${sensor_box_x_proximal}" y="${sensor_box_y}" z="${sensor_box_z}"/>
-          </xacro:if>
-          <xacro:if value="${location == 'distal'}">
-            <xacro:cuboid_inertia m="${sensor_mass}" x="${sensor_box_x_distal}" y="${sensor_box_y}" z="${sensor_box_z}"/>
-          </xacro:if>
+        <xacro:if value="${location == 'proximal'}">
+          <xacro:cuboid_inertia m="${sensor_mass}" x="${sensor_box_x_proximal}" y="${sensor_box_y}" z="${sensor_box_z}"/>
+        </xacro:if>
+        <xacro:if value="${location == 'distal'}">
+          <xacro:cuboid_inertia m="${sensor_mass}" x="${sensor_box_x_distal}" y="${sensor_box_y}" z="${sensor_box_z}"/>
+        </xacro:if>
       </inertial>
       <collision>

Commit message: Move pad collison boxes to parent element

File: reflex_stack/simulation/description/urdf/reflex/reflex.urdf.xacro (robot description, xacro)
@@ -68,4 +68,59 @@
     </link>
   </xacro:macro>
+  <xacro:property name="proximal_pad_box_x" value="0.016"/>
+  <xacro:property name="proximal_pad_box_y" value="0.020"/>
+  <xacro:property name="proximal_pad_box_z" value="0.052"/>
+  <xacro:macro name="proximal_pad" params="finger_id">
+    <link name="proximal_${finger_id}_pad">
+      <visual>
+        <origin xyz="-0.008 0.014 -0.002" rpy="${pi/2} ${pi/2} 0" />
+        <geometry>
+          <mesh filename="${mesh_path}/proximal_pad.STL"/>
+        </geometry>
+        <material name="dark_grey"/>
+      </visual>
+      <inertial>
+        <origin xyz="0 0.004 -0.035" rpy="0 0 0"/>
+        <mass value="${proximal_pad_mass}"/>
+        <xacro:cuboid_inertia m="${proximal_pad_mass}" x="${proximal_pad_box_x}" y="${proximal_pad_box_y}" z="${proximal_pad_box_z}"/>
+      </inertial>
+      <xacro:unless value="$(arg simplify_collisions)">
+        <collision>
+          <origin xyz="-0.008 0.014 -0.002" rpy="${pi/2} ${pi/2} 0"/>
+          <geometry>
+            <mesh filename="${mesh_path}/proximal_pad_coll.STL"/>
+          </geometry>
+        </collision>
+      </xacro:unless>
+    </link>
+  </xacro:macro>
+  <xacro:property name="distal_pad_box_x" value="${proximal_pad_box_x}"/>
+  <xacro:property name="distal_pad_box_y" value="0.018"/>
+  <xacro:property name="distal_pad_box_z" value="0.0385"/>
+  <xacro:macro name="distal_pad" params="finger_id">
+    <link name="distal_${finger_id}_pad">
+      <visual>
+        <!-- setting these xyz values by eye as transformations get too complex -->
+        <origin xyz="-0.008 0.0155 0.076" rpy="${pi/2} ${pi/2} 0"/>
+        <geometry>
+          <mesh filename="${mesh_path}/distal_pad.STL"/>
+        </geometry>
+        <material name="dark_grey"/>
+      </visual>
+      <inertial>
+        <origin xyz="0 ${distal_pad_box_y/2-0.002} ${-distal_pad_box_z/2+0.0005}" rpy="0 0 0"/>
+        <mass value="${distal_pad_mass}"/>
+        <xacro:cuboid_inertia m="${distal_pad_mass}" x="${distal_pad_box_x}" y="${distal_pad_box_y}" z="${distal_pad_box_z}"/>
+      </inertial>
+      <xacro:unless value="$(arg simplify_collisions)">
+        <collision>
+          <origin xyz="-0.008 0.0155 0.076" rpy="${pi/2} ${pi/2} 0"/>
+          <geometry>
+            <mesh filename="${mesh_path}/distal_pad_coll.STL"/>
+          </geometry>
+        </collision>
+      </xacro:unless>
+    </link>
+  </xacro:macro>
   <!-- approx length, height and width of a cuboid surrounding the link -->
   <xacro:property name="proximal_link_box_x" value="0.071"/>
@@ -86,12 +141,19 @@
         <xacro:cuboid_inertia m="${proximal_link_mass}" x="${proximal_link_box_x}" y="${proximal_link_box_y}" z="${proximal_link_box_z}"/>
       </inertial>
-      <xacro:unless value="$(arg simplify_collisions)">
-        <collision>
+      <collision>
+        <xacro:unless value="$(arg simplify_collisions)">
           <origin xyz="-0.011 0.007 0.011" rpy="${pi} 0 0"/>
           <geometry>
             <mesh filename="${mesh_path}/proximal_coll.STL"/>
           </geometry>
-        </collision>
-      </xacro:unless>
+        </xacro:unless>
+        <!-- attaching the collision box of pad here because libgazebo_ros_bumper only works if the collision box is on this parent link -->
+        <xacro:if value="$(arg simplify_collisions)">
+          <origin xyz="${proximal_link_box_x/2+0.001} 0 0.004" rpy="${pi/2} 0 -${pi/2}"/>
+          <geometry>
+            <box size="${proximal_pad_box_x} ${proximal_pad_box_y} ${proximal_pad_box_z}"/>
+          </geometry>
+        </xacro:if>
+      </collision>
     </link>
   </xacro:macro>
@@ -114,74 +176,14 @@
         <xacro:cuboid_inertia m="${distal_link_mass}" x="${distal_link_box_x}" y="${distal_link_box_y}" z="${distal_link_box_z}"/>
       </inertial>
-      <xacro:unless value="$(arg simplify_collisions)">
-        <collision>
-          <origin xyz="${-0.077-flex_link_box_x/2} 0.007 ${0.007+flex_link_box_z/2}" rpy="${pi} 0 0"/>
-          <geometry>
-            <mesh filename="${mesh_path}/distal_coll.STL"/>
-          </geometry>
-        </collision>
-      </xacro:unless>
-    </link>
-  </xacro:macro>
-  <xacro:property name="proximal_pad_box_x" value="0.016"/>
-  <xacro:property name="proximal_pad_box_y" value="0.020"/>
-  <xacro:property name="proximal_pad_box_z" value="0.052"/>
-  <xacro:macro name="proximal_pad" params="finger_id">
-    <link name="proximal_${finger_id}_pad">
-      <visual>
-        <origin xyz="-0.008 0.014 -0.002" rpy="${pi/2} ${pi/2} 0" />
-        <geometry>
-          <mesh filename="${mesh_path}/proximal_pad.STL"/>
-        </geometry>
-        <material name="dark_grey"/>
-      </visual>
-      <inertial>
-        <origin xyz="0 0.004 -0.035" rpy="0 0 0"/>
-        <mass value="${proximal_pad_mass}"/>
-        <xacro:cuboid_inertia m="${proximal_pad_mass}" x="${proximal_pad_box_x}" y="${proximal_pad_box_y}" z="${proximal_pad_box_z}"/>
-      </inertial>
       <collision>
         <xacro:unless value="$(arg simplify_collisions)">
-          <origin xyz="-0.008 0.014 -0.002" rpy="${pi/2} ${pi/2} 0"/>
-          <geometry>
-            <mesh filename="${mesh_path}/proximal_pad_coll.STL"/>
+          <origin xyz="${-0.077-flex_link_box_x/2} 0.007 ${0.007+flex_link_box_z/2}" rpy="${pi} 0 0"/>
+          <geometry>
+            <mesh filename="${mesh_path}/distal_coll.STL"/>
           </geometry>
         </xacro:unless>
+        <!-- attaching the collision box of pad here because libgazebo_ros_bumper only works if the collision box is on this parent link -->
         <xacro:if value="$(arg simplify_collisions)">
-          <origin xyz="0 0.004 -0.035" rpy="0 0 0"/>
-          <geometry>
-            <box size="${proximal_pad_box_x} ${proximal_pad_box_y} ${proximal_pad_box_z}"/>
-          </geometry>
-        </xacro:if>
-      </collision>
-    </link>
-  </xacro:macro>
-  <xacro:property name="distal_pad_box_x" value="${proximal_pad_box_x}"/>
-  <xacro:property name="distal_pad_box_y" value="0.018"/>
-  <xacro:property name="distal_pad_box_z" value="0.0385"/>
-  <xacro:macro name="distal_pad" params="finger_id">
-    <link name="distal_${finger_id}_pad">
-      <visual>
-        <!-- setting these xyz values by eye as transformations get too complex -->
-        <origin xyz="-0.008 0.0155 0.076" rpy="${pi/2} ${pi/2} 0"/>
-        <geometry>
-          <mesh filename="${mesh_path}/distal_pad.STL"/>
-        </geometry>
-        <material name="dark_grey"/>
-      </visual>
-      <inertial>
-        <origin xyz="0 ${distal_pad_box_y/2-0.002} ${-distal_pad_box_z/2+0.0005}" rpy="0 0 0"/>
-        <mass value="${distal_pad_mass}"/>
-        <xacro:cuboid_inertia m="${distal_pad_mass}" x="${distal_pad_box_x}" y="${distal_pad_box_y}" z="${distal_pad_box_z}"/>
-      </inertial>
-      <collision>
-        <xacro:unless value="$(arg simplify_collisions)">
-          <origin xyz="-0.008 0.0155 0.076" rpy="${pi/2} ${pi/2} 0"/>
-          <geometry>
-            <mesh filename="${mesh_path}/distal_pad_coll.STL"/>
-          </geometry>
-        </xacro:unless>
-        <xacro:if value="$(arg simplify_collisions)">
-          <origin xyz="0 ${distal_pad_box_y/2-0.002} ${-distal_pad_box_z/2+0.0005}" rpy="0 0 0"/>
+          <origin xyz="${distal_pad_box_x+0.0025} 0 0.0065" rpy="${pi/2} 0 -${pi/2}"/>
           <geometry>
             <box size="${distal_pad_box_x} ${distal_pad_box_y} ${distal_pad_box_z}"/>
