Commit message: Revert changes on pad back

File: reflex_stack/simulation/description/urdf/reflex/reflex.urdf.xacro (robot description, xacro)
@@ -68,59 +68,4 @@
     </link>
   </xacro:macro>
-  <xacro:property name="proximal_pad_box_x" value="0.016"/>
-  <xacro:property name="proximal_pad_box_y" value="0.020"/>
-  <xacro:property name="proximal_pad_box_z" value="0.052"/>
-  <xacro:macro name="proximal_pad" params="finger_id">
-    <link name="proximal_${finger_id}_pad">
-      <visual>
-        <origin xyz="-0.008 0.014 -0.002" rpy="${pi/2} ${pi/2} 0" />
-        <geometry>
-          <mesh filename="${mesh_path}/proximal_pad.STL"/>
-        </geometry>
-        <material name="dark_grey"/>
-      </visual>
-      <inertial>
-        <origin xyz="0 0.004 -0.035" rpy="0 0 0"/>
-        <mass value="${proximal_pad_mass}"/>
-        <xacro:cuboid_inertia m="${proximal_pad_mass}" x="${proximal_pad_box_x}" y="${proximal_pad_box_y}" z="${proximal_pad_box_z}"/>
-      </inertial>
-      <xacro:unless value="$(arg simplify_collisions)">
-        <collision>
-          <origin xyz="-0.008 0.014 -0.002" rpy="${pi/2} ${pi/2} 0"/>
-          <geometry>
-            <mesh filename="${mesh_path}/proximal_pad_coll.STL"/>
-          </geometry>
-        </collision>
-      </xacro:unless>
-    </link>
-  </xacro:macro>
-  <xacro:property name="distal_pad_box_x" value="${proximal_pad_box_x}"/>
-  <xacro:property name="distal_pad_box_y" value="0.018"/>
-  <xacro:property name="distal_pad_box_z" value="0.0385"/>
-  <xacro:macro name="distal_pad" params="finger_id">
-    <link name="distal_${finger_id}_pad">
-      <visual>
-        <!-- setting these xyz values by eye as transformations get too complex -->
-        <origin xyz="-0.008 0.0155 0.076" rpy="${pi/2} ${pi/2} 0"/>
-        <geometry>
-          <mesh filename="${mesh_path}/distal_pad.STL"/>
-        </geometry>
-        <material name="dark_grey"/>
-      </visual>
-      <inertial>
-        <origin xyz="0 ${distal_pad_box_y/2-0.002} ${-distal_pad_box_z/2+0.0005}" rpy="0 0 0"/>
-        <mass value="${distal_pad_mass}"/>
-        <xacro:cuboid_inertia m="${distal_pad_mass}" x="${distal_pad_box_x}" y="${distal_pad_box_y}" z="${distal_pad_box_z}"/>
-      </inertial>
-      <xacro:unless value="$(arg simplify_collisions)">
-        <collision>
-          <origin xyz="-0.008 0.0155 0.076" rpy="${pi/2} ${pi/2} 0"/>
-          <geometry>
-            <mesh filename="${mesh_path}/distal_pad_coll.STL"/>
-          </geometry>
-        </collision>
-      </xacro:unless>
-    </link>
-  </xacro:macro>
   <!-- approx length, height and width of a cuboid surrounding the link -->
   <xacro:property name="proximal_link_box_x" value="0.071"/>
@@ -141,19 +86,12 @@
         <xacro:cuboid_inertia m="${proximal_link_mass}" x="${proximal_link_box_x}" y="${proximal_link_box_y}" z="${proximal_link_box_z}"/>
       </inertial>
-      <collision>
-        <xacro:unless value="$(arg simplify_collisions)">
+      <xacro:unless value="$(arg simplify_collisions)">
+        <collision>
           <origin xyz="-0.011 0.007 0.011" rpy="${pi} 0 0"/>
           <geometry>
             <mesh filename="${mesh_path}/proximal_coll.STL"/>
           </geometry>
-        </xacro:unless>
-        <!-- attaching the collision box of pad here because libgazebo_ros_bumper only works if the collision box is on this parent link -->
-        <xacro:if value="$(arg simplify_collisions)">
-          <origin xyz="${proximal_link_box_x/2+0.001} 0 0.004" rpy="${pi/2} 0 -${pi/2}"/>
-          <geometry>
-            <box size="${proximal_pad_box_x} ${proximal_pad_box_y} ${proximal_pad_box_z}"/>
-          </geometry>
-        </xacro:if>
-      </collision>
+        </collision>
+      </xacro:unless>
     </link>
   </xacro:macro>
@@ -176,14 +114,74 @@
         <xacro:cuboid_inertia m="${distal_link_mass}" x="${distal_link_box_x}" y="${distal_link_box_y}" z="${distal_link_box_z}"/>
       </inertial>
+      <xacro:unless value="$(arg simplify_collisions)">
+        <collision>
+          <origin xyz="${-0.077-flex_link_box_x/2} 0.007 ${0.007+flex_link_box_z/2}" rpy="${pi} 0 0"/>
+          <geometry>
+            <mesh filename="${mesh_path}/distal_coll.STL"/>
+          </geometry>
+        </collision>
+      </xacro:unless>
+    </link>
+  </xacro:macro>
+  <xacro:property name="proximal_pad_box_x" value="0.016"/>
+  <xacro:property name="proximal_pad_box_y" value="0.020"/>
+  <xacro:property name="proximal_pad_box_z" value="0.052"/>
+  <xacro:macro name="proximal_pad" params="finger_id">
+    <link name="proximal_${finger_id}_pad">
+      <visual>
+        <origin xyz="-0.008 0.014 -0.002" rpy="${pi/2} ${pi/2} 0" />
+        <geometry>
+          <mesh filename="${mesh_path}/proximal_pad.STL"/>
+        </geometry>
+        <material name="dark_grey"/>
+      </visual>
+      <inertial>
+        <origin xyz="0 0.004 -0.035" rpy="0 0 0"/>
+        <mass value="${proximal_pad_mass}"/>
+        <xacro:cuboid_inertia m="${proximal_pad_mass}" x="${proximal_pad_box_x}" y="${proximal_pad_box_y}" z="${proximal_pad_box_z}"/>
+      </inertial>
       <collision>
         <xacro:unless value="$(arg simplify_collisions)">
-          <origin xyz="${-0.077-flex_link_box_x/2} 0.007 ${0.007+flex_link_box_z/2}" rpy="${pi} 0 0"/>
-          <geometry>
-            <mesh filename="${mesh_path}/distal_coll.STL"/>
+          <origin xyz="-0.008 0.014 -0.002" rpy="${pi/2} ${pi/2} 0"/>
+          <geometry>
+            <mesh filename="${mesh_path}/proximal_pad_coll.STL"/>
           </geometry>
         </xacro:unless>
-        <!-- attaching the collision box of pad here because libgazebo_ros_bumper only works if the collision box is on this parent link -->
         <xacro:if value="$(arg simplify_collisions)">
-          <origin xyz="${distal_pad_box_x+0.0025} 0 0.0065" rpy="${pi/2} 0 -${pi/2}"/>
+          <origin xyz="0 0.004 -0.036" rpy="0 0 0"/>
+          <geometry>
+            <box size="${proximal_pad_box_x} ${proximal_pad_box_y} ${proximal_pad_box_z}"/>
+          </geometry>
+        </xacro:if>
+      </collision>
+    </link>
+  </xacro:macro>
+  <xacro:property name="distal_pad_box_x" value="${proximal_pad_box_x}"/>
+  <xacro:property name="distal_pad_box_y" value="0.018"/>
+  <xacro:property name="distal_pad_box_z" value="0.0385"/>
+  <xacro:macro name="distal_pad" params="finger_id">
+    <link name="distal_${finger_id}_pad">
+      <visual>
+        <!-- setting these xyz values by eye as transformations get too complex -->
+        <origin xyz="-0.008 0.0155 0.076" rpy="${pi/2} ${pi/2} 0"/>
+        <geometry>
+          <mesh filename="${mesh_path}/distal_pad.STL"/>
+        </geometry>
+        <material name="dark_grey"/>
+      </visual>
+      <inertial>
+        <origin xyz="0 ${distal_pad_box_y/2-0.002} ${-distal_pad_box_z/2+0.0005}" rpy="0 0 0"/>
+        <mass value="${distal_pad_mass}"/>
+        <xacro:cuboid_inertia m="${distal_pad_mass}" x="${distal_pad_box_x}" y="${distal_pad_box_y}" z="${distal_pad_box_z}"/>
+      </inertial>
+      <collision>
+        <xacro:unless value="$(arg simplify_collisions)">
+          <origin xyz="-0.008 0.0155 0.076" rpy="${pi/2} ${pi/2} 0"/>
+          <geometry>
+            <mesh filename="${mesh_path}/distal_pad_coll.STL"/>
+          </geometry>
+        </xacro:unless>
+        <xacro:if value="$(arg simplify_collisions)">
+          <origin xyz="0 ${distal_pad_box_y/2-0.002} ${-distal_pad_box_z/2+0.0005}" rpy="0 0 0"/>
           <geometry>
             <box size="${distal_pad_box_x} ${distal_pad_box_y} ${distal_pad_box_z}"/>

Commit message: Change inertia box position

File: reflex_stack/simulation/description/urdf/reflex/reflex.urdf.xacro (robot description, xacro)
@@ -137,5 +137,5 @@
       </visual>
       <inertial>
-        <origin xyz="0 0.004 -0.035" rpy="0 0 0"/>
+        <origin xyz="0 0.004 -0.036" rpy="0 0 0"/>
         <mass value="${proximal_pad_mass}"/>
         <xacro:cuboid_inertia m="${proximal_pad_mass}" x="${proximal_pad_box_x}" y="${proximal_pad_box_y}" z="${proximal_pad_box_z}"/>

Commit message: Change height of collision element for pad

File: reflex_stack/simulation/description/urdf/reflex/reflex.urdf.xacro (robot description, xacro)
@@ -221,5 +221,5 @@
   <!-- approx length, height and width of a cuboid surrounding the link -->
   <xacro:property name="shell_box_x" value="0.13"/>
-  <xacro:property name="shell_box_y" value="0.09"/>
+  <xacro:property name="shell_box_y" value="0.084"/>
   <xacro:property name="shell_box_z" value="0.07"/>
   <xacro:property name="shell_x_offset" value="0.01"/>
@@ -273,7 +273,7 @@
         </xacro:unless>
         <xacro:if value="$(arg simplify_collisions)">
-          <origin xyz="0 ${pad_box_y/2} ${pad_x_offset}" rpy="0 0 0"/>
-          <geometry>
-            <box size="${shell_box_y} ${pad_box_y} ${shell_box_x}"/>
+          <origin xyz="0 -0.021 ${pad_x_offset}" rpy="0 0 0"/>
+          <geometry>
+            <box size="${shell_box_y} ${shell_box_y} ${shell_box_x}"/>
           </geometry>
         </xacro:if>

Commit message: Update urdf

File: reflex_stack/simulation/description/urdf/reflex/reflex.urdf.xacro (robot description, xacro)
@@ -412,12 +412,49 @@
     </joint>
   </xacro:macro>
-  <xacro:macro name="flex_to_distal" params="finger_id">
+  <!-- dummy links for revolute joints to latch on to -->
+  <xacro:property name="dummy_link_mass" value="0.01"/>
+  <xacro:property name="dummy_link_size" value="0.01"/>
+  <xacro:property name="dummy_joint_lim_max" value="3"/>
+  <xacro:property name="dummy_joint_lim_min" value="-3"/>
+  <xacro:property name="dummy_damping" value="0.01"/>
+  <xacro:property name="dummy_stiffness" value="0.01"/>
+  <xacro:property name="dummy_friction" value="0.01"/>
+  <xacro:macro name="dummy_link" params="finger_id dummy_link_id">
+    <link name="dummy_link_f${finger_id}_id${dummy_link_id}">
+      <inertial>
+        <origin rpy="0 0 0" xyz="0 0 0"/>
+        <mass value="${dummy_link_mass}"/>
+        <xacro:cuboid_inertia m="${dummy_link_mass}" x="${dummy_link_size}" y="${dummy_link_size}" z="${dummy_link_size}"/>
+      </inertial>
+    </link>
+  </xacro:macro>
+  <xacro:macro name="flex_to_distal" params="finger_id dummy_link_id">
     <joint name="flex_to_distal_${finger_id}" type="revolute">
       <origin xyz="${flex_link_box_x} 0 0" rpy="0 0 0"/>
       <parent link="finger_${finger_id}_flex_link"/>
-      <child link="distal_${finger_id}"/>
+      <child link="dummy_link_f${finger_id}_id${dummy_link_id}"/>
       <axis xyz="0 -1 0"/>
       <dynamics damping="${flex_joints_damping}" friction="${flex_joints_friction}"/>
       <limit effort="${flex_joints_effort}" lower="0.0" upper="${pi/6}" velocity="${flex_joints_velocity}"/>
+    </joint>
+  </xacro:macro>
+  <xacro:macro name="dummy_to_dummy" params="finger_id parent_dummy_id child_dummy_id">
+    <joint name="dummy_to_dummy_${finger_id}" type="revolute">
+      <origin xyz="0 0 0" rpy="0 0 0"/>
+      <parent link="dummy_link_f${finger_id}_id${parent_dummy_id}"/>
+      <child link="dummy_link_f${finger_id}_id${child_dummy_id}"/>
+      <axis xyz="1 0 0"/>
+      <dynamics damping="${dummy_damping}" friction="${dummy_friction}" spring_stiffness="${dummy_stiffness}"/>
+      <limit effort="1" velocity="0.2" lower="${dummy_joint_lim_min}" upper="${dummy_joint_lim_max}"/>
+    </joint>
+  </xacro:macro>
+  <xacro:macro name="dummy_to_distal" params="finger_id parent_dummy_id">
+    <joint name="dummy_to_distal_${finger_id}" type="revolute">
+      <origin xyz="0 0 0" rpy="0 0 0"/>
+      <parent link="dummy_link_f${finger_id}_id${parent_dummy_id}"/>
+      <child link="distal_${finger_id}"/>
+      <axis xyz="0 0 1"/>
+      <dynamics damping="${dummy_damping}" friction="${dummy_friction}" spring_stiffness="${dummy_stiffness}"/>
+      <limit effort="1" velocity="0.2" lower="${dummy_joint_lim_min}" upper="${dummy_joint_lim_max}"/>
     </joint>
   </xacro:macro>
@@ -444,5 +481,9 @@
     <xacro:proximal_to_flex finger_id="${id}"/>
     <xacro:flex_link finger_id="${id}"/>
-    <xacro:flex_to_distal finger_id="${id}"/>
+    <xacro:flex_to_distal finger_id="${id}" dummy_link_id="1"/>
+    <xacro:dummy_link finger_id="${id}" dummy_link_id="1"/>
+    <xacro:dummy_to_dummy finger_id="${id}" parent_dummy_id="1" child_dummy_id="2"/>
+    <xacro:dummy_link finger_id="${id}" dummy_link_id="2"/>
+    <xacro:dummy_to_distal finger_id="${id}" parent_dummy_id="2"/>
     <xacro:distal_link finger_id="${id}"/>
     <xacro:distal_to_pad finger_id="${id}"/>
