Commit message: Add inertia calculation

File: reflex_stack/simulation/description/urdf/environment/box.urdf.xacro (robot description, xacro)
@@ -3,9 +3,9 @@
     <!-- arguments -->
     <xacro:arg name="box_mass" default="0.2"/>
-    <xacro:arg name="box_inertia" default="0.0006"/>
     <xacro:arg name="box_x" default="0.08"/>
     <xacro:arg name="box_y" default="0.08"/>
     <xacro:arg name="box_z" default="0.08"/>
     <xacro:property name="link_name" value="box_link"/>
+    <xacro:include filename="$(find description)/urdf/xacro_macros/inertia_tensors.xacro"/>
     <link name="${link_name}">
         <visual>
@@ -24,5 +24,5 @@
             <origin xyz="0 0 0" rpy="0 0 0"/>
             <mass value="$(arg box_mass)"/>
-            <inertia ixx="$(arg box_inertia)" ixy="0" ixz="0" iyy="$(arg box_inertia)" iyz="0" izz="$(arg box_inertia)" />
+            <xacro:cuboid_inertia m="$(arg box_mass)" x="$(arg box_x)" y="$(arg box_y)" z="$(arg box_z)" />
         </inertial>
     </link>

File: reflex_stack/simulation/description/urdf/environment/cylinder.urdf.xacro (robot description, xacro)
@@ -2,9 +2,9 @@
 <robot xmlns:xacro="http://ros.org/wiki/xacro" name="cylinder">
     <!-- arguments -->
-    <xacro:arg name="cylinder_mass" default="0.2"/>
-    <xacro:arg name="cylinder_inertia" default="0.0006"/>
-    <xacro:arg name="cylinder_radius" default="0.08"/>
-    <xacro:arg name="cylinder_length" default="0.08"/>
+    <xacro:arg name="cylinder_mass" default="0.5"/>
+    <xacro:arg name="cylinder_radius" default="0.04"/>
+    <xacro:arg name="cylinder_length" default="0.15"/>
     <xacro:property name="link_name" value="cylinder_link"/>
+    <xacro:include filename="$(find description)/urdf/xacro_macros/inertia_tensors.xacro"/>
     <link name="${link_name}">
         <visual>
@@ -23,5 +23,5 @@
             <origin xyz="0 0 0" rpy="0 0 0"/>
             <mass value="$(arg cylinder_mass)"/>
-            <inertia ixx="$(arg cylinder_inertia)" ixy="0" ixz="0" iyy="$(arg cylinder_inertia)" iyz="0" izz="$(arg cylinder_inertia)" />
+            <xacro:cylinder_inertia m="$(arg cylinder_mass)" r="$(arg cylinder_radius)" h="$(arg cylinder_length)"/>
         </inertial>
     </link>

File: reflex_stack/simulation/description/urdf/environment/sphere.urdf.xacro (robot description, xacro)
@@ -3,7 +3,7 @@
     <!-- arguments -->
     <xacro:arg name="sphere_mass" default="0.2"/>
-    <xacro:arg name="sphere_inertia" default="0.0006"/>
     <xacro:arg name="sphere_radius" default="0.08"/>
     <xacro:property name="link_name" value="sphere_link"/>
+    <xacro:include filename="$(find description)/urdf/xacro_macros/inertia_tensors.xacro"/>
     <link name="${link_name}">
         <visual>
@@ -22,5 +22,5 @@
             <origin xyz="0 0 0" rpy="0 0 0"/>
             <mass value="$(arg sphere_mass)"/>
-            <inertia ixx="$(arg sphere_inertia)" ixy="0" ixz="0" iyy="$(arg sphere_inertia)" iyz="0" izz="$(arg sphere_inertia)" />
+            <xacro:sphere_inertia m="$(arg sphere_mass)" r="$(arg sphere_radius)" />
         </inertial>
     </link>
